File: hardware/analog/electro_chemistry/electrochem_board_v1/electrochem_board_v1/mcu_ifc.sch (KiCad schematic (older format))
At the start: 0 parts

Commit message: started Electrochemistry board
Parts:
- added J?: Conn_01x20_Male, symbol Connector:Conn_01x20_Male
Changed lines of the file:
@@
 $Descr A4 11693 8268
 encoding utf-8
-Sheet 1 8
+Sheet 2 9
 Title ""
 Date ""
@@
 Comment4 ""
 $EndDescr
+$Comp
+L Connector:Conn_01x20_Male J?
+U 1 1 6096EB1E
+P 3500 3800
+F 0 "J?" H 3608 4881 50  0000 C CNN
+F 1 "Conn_01x20_Male" H 3608 4790 50  0000 C CNN
+F 2 "" H 3500 3800 50  0001 C CNN
+F 3 "~" H 3500 3800 50  0001 C CNN
+	1    3500 3800
+	1    0    0    -1
+$EndComp
 $EndSCHEMATC
