File: hardware/analog/electro_chemistry/electrochem_board_v1/electrochem_board_v1/asense.sch (KiCad schematic (older format))
At the start: 0 parts

Commit message: started Electrochemistry board
Parts:
- added U?: INA181, Package_TO_SOT_SMD:SOT-23-6, symbol Amplifier_Current:INA181
Changed lines of the file:
@@
 $Descr A4 11693 8268
 encoding utf-8
-Sheet 1 9
+Sheet 8 9
 Title ""
 Date ""
@@
 Comment4 ""
 $EndDescr
+$Comp
+L Amplifier_Current:INA181 U?
+U 1 1 6096FFE7
+P 4750 3350
+F 0 "U?" H 5094 3396 50  0000 L CNN
+F 1 "INA181" H 5094 3305 50  0000 L CNN
+F 2 "Package_TO_SOT_SMD:SOT-23-6" H 4800 3400 50  0001 C CNN
+F 3 "http://www.ti.com/lit/ds/symlink/ina181.pdf" H 4900 3500 50  0001 C CNN
+	1    4750 3350
+	1    0    0    -1
+$EndComp
 $EndSCHEMATC
