File: hardware/analog/electro_chemistry/electrochem_board_v1/electrochem_board_v1/psu_ifc.sch (KiCad schematic (older format))
At the start: 0 parts

Commit message: started Electrochemistry board
Parts:
- added J?: ATX-24, symbol Connector:ATX-24
Connections:
- new net: J?.1 (+3.3V), J?.12 (+3.3V), J?.13 (+3.3V), J?.2 (+3.3V)
- new net: J?.10 (+12V), J?.11 (+12V)
- new net: J?.15 (GND), J?.17 (GND), J?.18 (GND), J?.19 (GND), J?.24 (GND), J?.3 (GND), J?.5 (GND), J?.7 (GND)
- new net: J?.21 (+5V), J?.22 (+5V), J?.23 (+5V), J?.4 (+5V), J?.6 (+5V)
Changed lines of the file:
@@
 $Descr A4 11693 8268
 encoding utf-8
-Sheet 1 9
+Sheet 3 9
 Title ""
 Date ""
@@
 Comment4 ""
 $EndDescr
+$Comp
+L Connector:ATX-24 J?
+U 1 1 60970A62
+P 3900 3300
+F 0 "J?" H 3900 3967 50  0000 C CNN
+F 1 "ATX-24" H 3900 3876 50  0000 C CNN
+F 2 "" H 3900 3200 50  0001 C CNN
+F 3 "https://www.intel.com/content/dam/www/public/us/en/documents/guides/power-supply-design-guide-june.pdf#page=33" H 6300 2750 50  0001 C CNN
+	1    3900 3300
+	1    0    0    -1
+$EndComp
 $EndSCHEMATC
