File: hardware/fpga/ice40std/ice40up5brdV1/ice40up5brdV1/nand.sch (KiCad schematic (older format))
At the start: 0 parts

Commit message: usb => mcu => ice40 fpga => NAND flash bridge started
Parts:
- added C1: 0.1uF, Capacitor_SMD:C_0402_1005Metric, symbol Device:C
- added C2: 4.7uF, Capacitor_SMD:C_0402_1005Metric, symbol Device:C
- added J2: Conn_01x20_Male, Connector_PinSocket_2.54mm:PinSocket_1x20_P2.54mm_Horizontal, symbol Connector:Conn_01x20_Male
- added U1: MT29F1G08ABAEAWP, Package_SO:TSOP-I-48_18.4x12mm_P0.5mm, symbol digital:MT29F1G08ABAEAWP
Connections:
- net labels added: +3V3, ALE, CE, CLE, D0, D1, D2, D3, D4, D5, D6, D7, GND, RE, WE, WP
- wire segments 0 -> 38
