File: hardware/fpga/ice40std/ice40up5brdV1/ice40up5brdV1/ice40up5brdV1.kicad_pcb (KiCad board)
At the start: 2 copper layers, 93.1 x 60.2 mm, 59 parts, among them J1 Conn_01x20_Male, J2 Conn_01x20_Female, J3 Conn_01x06_Male, SW1 SW_Push, SW2 SW_Push, SW3 SW_Push, U1 ICE40UP5K-SG48ITR, U2 LTC3406ES5, U3 LTC3406ES5, U4 AT25SF081-SSHD-X, U5 ATSAMD11D14A-M, U6 MT29F1G08ABAEAWP, X1 ASE-xxxMHz, X2 USBFCI_10103594_MILL

Commit message: ice40qfn restarted
Parts:
- removed C16: 0.1uF, Capacitor_SMD:C_0402_1005Metric
- removed C17: 4.7uF, Capacitor_SMD:C_0402_1005Metric
- removed R17: R, Resistor_SMD:R_0402_1005Metric
- removed U6: MT29F1G08ABAEAWP, Package_SO:TSOP-I-48_18.4x12mm_P0.5mm
- removed X2: USBFCI_10103594_MILL, kifootp:FCI_10103594_MILL
- added J4: Conn_01x04_Male, Connector_PinHeader_2.54mm:PinHeader_1x04_P2.54mm_Horizontal, F.Cu at (60.4, 107.3)
- added J5: Conn_01x04_Male, Connector_PinHeader_2.54mm:PinHeader_1x04_P2.54mm_Horizontal, F.Cu at (60.3, 93.7)
- J1, J2: footprint Connector_PinHeader_2.54mm:PinHeader_1x20_P2.54mm_Vertical -> Connector_PinHeader_2.54mm:PinHeader_1x20_P2.54mm_Horizontal
- moved J2 0.46 mm to (88.6, 133.9)
- moved J1 0.13 mm to (129.9, 83.2)
Routing:
- net +3V3: track 400.2 -> 338.7 mm
- net d0: track 37.4 -> 19.4 mm
- net d1: track 34.7 -> 18.3 mm
- net ale: track 44.2 -> 28.6 mm
- net d2: track 29.6 -> 15.8 mm
- net d3: track 27.7 -> 15.0 mm
- net d6: track 35.1 -> 22.5 mm
- net d5: track 31.0 -> 19.9 mm
- net d4: track 28.2 -> 17.5 mm
- net we: track 39.8 -> 29.6 mm, vias 1 -> 0
- net +5V: track 22.7 -> 32.8 mm
- net re: track 36.6 -> 26.8 mm, vias 0 -> 1
- net ce: track 31.9 -> 23.1 mm
- net d7: track 39.5 -> 31.3 mm, vias 1 -> 0
- net cle: track 36.0 -> 28.8 mm, vias 1 -> 0
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
Commit message: ice40qfn restarted
Parts:
- J1, J2: footprint Connector_PinHeader_2.54mm:PinHeader_1x20_P2.54mm_Horizontal -> Connector_PinHeader_2.54mm:PinHeader_1x20_P2.54mm_Vertical
- moved J5 7.42 mm to (60.6, 101.1), turned to 180 degrees
- moved J2 0.46 mm to (88.2, 134.0)
- moved J4 0.30 mm to (60.7, 107.2)
- moved J1 0.13 mm to (130.1, 83.2)
Routing:
- net +5V: track 32.8 -> 31.6 mm
- net ss: vias 2 -> 1
- net re: vias 1 -> 0
- net GND: vias 417 -> 418

Commit message: ice40qfn restarted
Parts:
- J4: footprint Connector_PinHeader_2.54mm:PinHeader_1x04_P2.54mm_Horizontal -> Connector_PinHeader_2.54mm:PinHeader_1x04_P2.54mm_Vertical
Changed lines of the file:
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@@
     (add_net we)
+  )
+  (module Connector_PinHeader_2.54mm:PinHeader_1x04_P2.54mm_Vertical (layer F.Cu)
+    (at 60.71 107.18)
+    (descr "Through hole straight pin header, 1x04, 2.54mm pitch, single row")
+    (tags "Through hole pin header THT 1x04 2.54mm single row")
+    (fp_text reference J4 (at 4.385 -2.27) (layer F.SilkS)
+      (effects (font (size 1 1) (thickness 0.15)))
+    )
+    (fp_text value Conn_01x04_Male (at 4.385 9.89) (layer F.Fab)
+      (effects (font (size 1 1) (thickness 0.15)))
+    )
+    (fp_text user %R (at 2.77 3.81 90) (layer F.Fab)
+      (effects (font (size 1 1) (thickness 0.15)))
+    )
+    (fp_line (start -0.635 -1.27) (end 1.27 -1.27) (layer F.Fab) (width 0.1))
+    (fp_line (start 1.27 -1.27) (end 1.27 8.89) (layer F.Fab) (width 0.1))
+    (fp_line (start 1.27 8.89) (end -1.27 8.89) (layer F.Fab) (width 0.1))
+    (fp_line (start -1.27 8.89) (end -1.27 -0.635) (layer F.Fab) (width 0.1))
+    (fp_line (start -1.27 -0.635) (end -0.635 -1.27) (layer F.Fab) (width 0.1))
+    (fp_line (start -1.33 8.95) (end 1.33 8.95) (layer F.SilkS) (width 0.12))
+    (fp_line (start -1.33 1.27) (end -1.33 8.95) (layer F.SilkS) (width 0.12))
+    (fp_line (start 1.33 1.27) (end 1.33 8.95) (layer F.SilkS) (width 0.12))
+    (fp_line (start -1.33 1.27) (end 1.33 1.27) (layer F.SilkS) (width 0.12))
+    (fp_line (start -1.33 0) (end -1.33 -1.33) (layer F.SilkS) (width 0.12))
+    (fp_line (start -1.33 -1.33) (end 0 -1.33) (layer F.SilkS) (width 0.12))
+    (fp_line (start -1.8 -1.8) (end -1.8 9.4) (layer F.CrtYd) (width 0.05))
+    (fp_line (start -1.8 9.4) (end 1.8 9.4) (layer F.CrtYd) (width 0.05))
+    (fp_line (start 1.8 9.4) (end 1.8 -1.8) (layer F.CrtYd) (width 0.05))
+    (fp_line (start 1.8 -1.8) (end -1.8 -1.8) (layer F.CrtYd) (width 0.05))
+    (pad 4 thru_hole oval (at 0 7.62) (size 1.7 1.7) (drill 1) (layers *.Cu *.Mask)
+      (net 1 GND))
+    (pad 3 thru_hole oval (at 0 5.08) (size 1.7 1.7) (drill 1) (layers *.Cu *.Mask)
+      (net 67 "Net-(J4-Pad3)"))
+    (pad 2 thru_hole oval (at 0 2.54) (size 1.7 1.7) (drill 1) (layers *.Cu *.Mask)
+      (net 68 "Net-(J4-Pad2)"))
+    (pad 1 thru_hole rect (at 0 0) (size 1.7 1.7) (drill 1) (layers *.Cu *.Mask)
+      (net 48 +5V))
+    (model ${KISYS3DMOD}/Connector_PinHeader_2.54mm.3dshapes/PinHeader_1x04_P2.54mm_Vertical.wrl
+      (at (xyz 0 0 0))
+      (scale (xyz 1 1 1))
+      (rotate (xyz 0 0 0))
+    )
   )
   (module Connector_PinHeader_2.54mm:PinHeader_1x04_P2.54mm_Horizontal (layer F.Cu)
@@
       (net 1 GND))
     (model ${KISYS3DMOD}/Connector_PinHeader_2.54mm.3dshapes/PinHeader_1x04_P2.54mm_Horizontal.wrl
-      (at (xyz 0 0 0))
-      (scale (xyz 1 1 1))
-      (rotate (xyz 0 0 0))
-    )
-  )
-  (module Connector_PinHeader_2.54mm:PinHeader_1x04_P2.54mm_Horizontal (layer F.Cu)
-    (at 60.71 107.18)
-    (descr "Through hole angled pin header, 1x04, 2.54mm pitch, 6mm pin length, single row")
-    (tags "Through hole angled pin header THT 1x04 2.54mm single row")
-    (fp_text reference J4 (at 4.385 -2.27) (layer F.SilkS)
-      (effects (font (size 1 1) (thickness 0.15)))
-    )
-    (fp_text value Conn_01x04_Male (at 4.385 9.89) (layer F.Fab)
-      (effects (font (size 1 1) (thickness 0.15)))
-    )
-    (fp_line (start 10.55 -1.8) (end -1.8 -1.8) (layer F.CrtYd) (width 0.05))
-    (fp_line (start 10.55 9.4) (end 10.55 -1.8) (layer F.CrtYd) (width 0.05))
-    (fp_line (start -1.8 9.4) (end 10.55 9.4) (layer F.CrtYd) (width 0.05))
-    (fp_line (start -1.8 -1.8) (end -1.8 9.4) (layer F.CrtYd) (width 0.05))
-    (fp_line (start -1.27 -1.27) (end 0 -1.27) (layer F.SilkS) (width 0.12))
-    (fp_line (start -1.27 0) (end -1.27 -1.27) (layer F.SilkS) (width 0.12))
-    (fp_line (start 1.042929 8) (end 1.44 8) (layer F.SilkS) (width 0.12))
-    (fp_line (start 1.042929 7.24) (end 1.44 7.24) (layer F.SilkS) (width 0.12))
-    (fp_line (start 10.1 8) (end 4.1 8) (layer F.SilkS) (width 0.12))
-    (fp_line (start 10.1 7.24) (end 10.1 8) (layer F.SilkS) (width 0.12))
-    (fp_line (start 4.1 7.24) (end 10.1 7.24) (layer F.SilkS) (width 0.12))
-    (fp_line (start 1.44 6.35) (end 4.1 6.35) (layer F.SilkS) (width 0.12))
-    (fp_line (start 1.042929 5.46) (end 1.44 5.46) (layer F.SilkS) (width 0.12))
-    (fp_line (start 1.042929 4.7) (end 1.44 4.7) (layer F.SilkS) (width 0.12))
-    (fp_line (start 10.1 5.46) (end 4.1 5.46) (layer F.SilkS) (width 0.12))
-    (fp_line (start 10.1 4.7) (end 10.1 5.46) (layer F.SilkS) (width 0.12))
-    (fp_line (start 4.1 4.7) (end 10.1 4.7) (layer F.SilkS) (width 0.12))
-    (fp_line (start 1.44 3.81) (end 4.1 3.81) (layer F.SilkS) (width 0.12))
-    (fp_line (start 1.042929 2.92) (end 1.44 2.92) (layer F.SilkS) (width 0.12))
-    (fp_line (start 1.042929 2.16) (end 1.44 2.16) (layer F.SilkS) (width 0.12))
-    (fp_line (start 10.1 2.92) (end 4.1 2.92) (layer F.SilkS) (width 0.12))
-    (fp_line (start 10.1 2.16) (end 10.1 2.92) (layer F.SilkS) (width 0.12))
-    (fp_line (start 4.1 2.16) (end 10.1 2.16) (layer F.SilkS) (width 0.12))
-    (fp_line (start 1.44 1.27) (end 4.1 1.27) (layer F.SilkS) (width 0.12))
-    (fp_line (start 1.11 0.38) (end 1.44 0.38) (layer F.SilkS) (width 0.12))
-    (fp_line (start 1.11 -0.38) (end 1.44 -0.38) (layer F.SilkS) (width 0.12))
-    (fp_line (start 4.1 0.28) (end 10.1 0.28) (layer F.SilkS) (width 0.12))
-    (fp_line (start 4.1 0.16) (end 10.1 0.16) (layer F.SilkS) (width 0.12))
-    (fp_line (start 4.1 0.04) (end 10.1 0.04) (layer F.SilkS) (width 0.12))
-    (fp_line (start 4.1 -0.08) (end 10.1 -0.08) (layer F.SilkS) (width 0.12))
-    (fp_line (start 4.1 -0.2) (end 10.1 -0.2) (layer F.SilkS) (width 0.12))
-    (fp_line (start 4.1 -0.32) (end 10.1 -0.32) (layer F.SilkS) (width 0.12))
-    (fp_line (start 10.1 0.38) (end 4.1 0.38) (layer F.SilkS) (width 0.12))
-    (fp_line (start 10.1 -0.38) (end 10.1 0.38) (layer F.SilkS) (width 0.12))
-    (fp_line (start 4.1 -0.38) (end 10.1 -0.38) (layer F.SilkS) (width 0.12))
-    (fp_line (start 4.1 -1.33) (end 1.44 -1.33) (layer F.SilkS) (width 0.12))
-    (fp_line (start 4.1 8.95) (end 4.1 -1.33) (layer F.SilkS) (width 0.12))
-    (fp_line (start 1.44 8.95) (end 4.1 8.95) (layer F.SilkS) (width 0.12))
-    (fp_line (start 1.44 -1.33) (end 1.44 8.95) (layer F.SilkS) (width 0.12))
-    (fp_line (start 4.04 7.94) (end 10.04 7.94) (layer F.Fab) (width 0.1))
-    (fp_line (start 10.04 7.3) (end 10.04 7.94) (layer F.Fab) (width 0.1))
-    (fp_line (start 4.04 7.3) (end 10.04 7.3) (layer F.Fab) (width 0.1))
-    (fp_line (start -0.32 7.94) (end 1.5 7.94) (layer F.Fab) (width 0.1))
-    (fp_line (start -0.32 7.3) (end -0.32 7.94) (layer F.Fab) (width 0.1))
-    (fp_line (start -0.32 7.3) (end 1.5 7.3) (layer F.Fab) (width 0.1))
-    (fp_line (start 4.04 5.4) (end 10.04 5.4) (layer F.Fab) (width 0.1))
-    (fp_line (start 10.04 4.76) (end 10.04 5.4) (layer F.Fab) (width 0.1))
-    (fp_line (start 4.04 4.76) (end 10.04 4.76) (layer F.Fab) (width 0.1))
-    (fp_line (start -0.32 5.4) (end 1.5 5.4) (layer F.Fab) (width 0.1))
-    (fp_line (start -0.32 4.76) (end -0.32 5.4) (layer F.Fab) (width 0.1))
-    (fp_line (start -0.32 4.76) (end 1.5 4.76) (layer F.Fab) (width 0.1))
-    (fp_line (start 4.04 2.86) (end 10.04 2.86) (layer F.Fab) (width 0.1))
-    (fp_line (start 10.04 2.22) (end 10.04 2.86) (layer F.Fab) (width 0.1))
-    (fp_line (start 4.04 2.22) (end 10.04 2.22) (layer F.Fab) (width 0.1))
-    (fp_line (start -0.32 2.86) (end 1.5 2.86) (layer F.Fab) (width 0.1))
-    (fp_line (start -0.32 2.22) (end -0.32 2.86) (layer F.Fab) (width 0.1))
-    (fp_line (start -0.32 2.22) (end 1.5 2.22) (layer F.Fab) (width 0.1))
-    (fp_line (start 4.04 0.32) (end 10.04 0.32) (layer F.Fab) (width 0.1))
-    (fp_line (start 10.04 -0.32) (end 10.04 0.32) (layer F.Fab) (width 0.1))
-    (fp_line (start 4.04 -0.32) (end 10.04 -0.32) (layer F.Fab) (width 0.1))
-    (fp_line (start -0.32 0.32) (end 1.5 0.32) (layer F.Fab) (width 0.1))
-    (fp_line (start -0.32 -0.32) (end -0.32 0.32) (layer F.Fab) (width 0.1))
-    (fp_line (start -0.32 -0.32) (end 1.5 -0.32) (layer F.Fab) (width 0.1))
-    (fp_line (start 1.5 -0.635) (end 2.135 -1.27) (layer F.Fab) (width 0.1))
-    (fp_line (start 1.5 8.89) (end 1.5 -0.635) (layer F.Fab) (width 0.1))
-    (fp_line (start 4.04 8.89) (end 1.5 8.89) (layer F.Fab) (width 0.1))
-    (fp_line (start 4.04 -1.27) (end 4.04 8.89) (layer F.Fab) (width 0.1))
-    (fp_line (start 2.135 -1.27) (end 4.04 -1.27) (layer F.Fab) (width 0.1))
-    (fp_text user %R (at 2.77 3.81 90) (layer F.Fab)
-      (effects (font (size 1 1) (thickness 0.15)))
-    )
-    (pad 1 thru_hole rect (at 0 0) (size 1.7 1.7) (drill 1) (layers *.Cu *.Mask)
-      (net 48 +5V))
-    (pad 2 thru_hole oval (at 0 2.54) (size 1.7 1.7) (drill 1) (layers *.Cu *.Mask)
-      (net 68 "Net-(J4-Pad2)"))
-    (pad 3 thru_hole oval (at 0 5.08) (size 1.7 1.7) (drill 1) (layers *.Cu *.Mask)
-      (net 67 "Net-(J4-Pad3)"))
-    (pad 4 thru_hole oval (at 0 7.62) (size 1.7 1.7) (drill 1) (layers *.Cu *.Mask)
-      (net 1 GND))
-    (model ${KISYS3DMOD}/Connector_PinHeader_2.54mm.3dshapes/PinHeader_1x04_P2.54mm_Horizontal.wrl

Commit message: ice40qfn restarted
Parts:
- removed J5: Conn_01x04_Male, Connector_PinHeader_2.54mm:PinHeader_1x04_P2.54mm_Horizontal
Routing:
- net +5V: track 31.6 -> 25.0 mm

Commit message: ice40qfn restarted: simplest design ready?
Routing:
- net d7: track 31.3 -> 23.5 mm
- net cle: track 28.8 -> 22.9 mm
- net we: track 29.6 -> 25.0 mm
- net +3V3: track 338.7 -> 335.2 mm, vias 2 -> 6
- net GND: vias 418 -> 437
- net +1V2: vias 3 -> 6
Other:
- board size 93.1 x 60.2 mm -> 75 x 59.9 mm
Changed lines of the file:
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@@
   (general
     (thickness 1.6)
-    (drawings 3)
-    (tracks 945)
+    (drawings 4)
+    (tracks 976)
     (zones 0)
     (modules 55)
@@
     )
   )
-  (gr_line (start 58.34 78.58) (end 149.52 78.55) (layer Edge.Cuts) (width 0.1))
-  (gr_line (start 58.25 138.75) (end 58.34 78.58) (layer Edge.Cuts) (width 0.1))
-  (gr_line (start 151.33 138.18) (end 58.25 138.75) (layer Edge.Cuts) (width 0.1))
+  (gr_line (start 133.31 78.42) (end 133.64 136.95) (layer Edge.Cuts) (width 0.1))
+  (gr_line (start 59.24 79.53) (end 133.31 78.42) (layer Edge.Cuts) (width 0.1))
+  (gr_line (start 58.66 138.32) (end 59.24 79.53) (layer Edge.Cuts) (width 0.1))
+  (gr_line (start 133.64 136.95) (end 58.66 138.32) (layer Edge.Cuts) (width 0.1))
   (via (at 113.88 106.16) (size 0.5) (drill 0.25) (layers F.Cu B.Cu) (net 1))
   (via (at 112.19 106.12) (size 0.5) (drill 0.25) (layers F.Cu B.Cu) (net 1))
@@
   (via (at 107.94 111.37) (size 0.5) (drill 0.25) (layers F.Cu B.Cu) (net 1))
   (via (at 110.25 111.05) (size 0.5) (drill 0.25) (layers F.Cu B.Cu) (net 1))
+  (via (at 114.08 113.31) (size 0.5) (drill 0.25) (layers F.Cu B.Cu) (net 1))
+  (via (at 116.24 113.41) (size 0.5) (drill 0.25) (layers F.Cu B.Cu) (net 1))
+  (via (at 117.25 112.33) (size 0.5) (drill 0.25) (layers F.Cu B.Cu) (net 1))
+  (via (at 116.2 110.97) (size 0.5) (drill 0.25) (layers F.Cu B.Cu) (net 1))
+  (via (at 116.39 116.04) (size 0.5) (drill 0.25) (layers F.Cu B.Cu) (net 1))
+  (via (at 117.6 114.67) (size 0.5) (drill 0.25) (layers F.Cu B.Cu) (net 1))
+  (via (at 118.61 113.38) (size 0.5) (drill 0.25) (layers F.Cu B.Cu) (net 1))
+  (via (at 122.51 110.64) (size 0.5) (drill 0.25) (layers F.Cu B.Cu) (net 1))
+  (via (at 120.82 109.25) (size 0.5) (drill 0.25) (layers F.Cu B.Cu) (net 1))
+  (via (at 124.69 112.84) (size 0.5) (drill 0.25) (layers F.Cu B.Cu) (net 1))
+  (via (at 123.35 111.51) (size 0.5) (drill 0.25) (layers F.Cu B.Cu) (net 1))
+  (via (at 118.5 106.81) (size 0.5) (drill 0.25) (layers F.Cu B.Cu) (net 1))
+  (via (at 119.98 108.39) (size 0.5) (drill 0.25) (layers F.Cu B.Cu) (net 1))
+  (via (at 121.52 105.88) (size 0.5) (drill 0.25) (layers F.Cu B.Cu) (net 1))
+  (via (at 122.19 106.81) (size 0.5) (drill 0.25) (layers F.Cu B.Cu) (net 1))
+  (via (at 123.77 108.52) (size 0.5) (drill 0.25) (layers F.Cu B.Cu) (net 1))
+  (via (at 125.58 108.95) (size 0.5) (drill 0.25) (layers F.Cu B.Cu) (net 1))
+  (via (at 125.08 107.54) (size 0.5) (drill 0.25) (layers F.Cu B.Cu) (net 1))
+  (via (at 125.83 107.47) (size 0.5) (drill 0.25) (layers F.Cu B.Cu) (net 1))
   (segment (start 114.38 114.84) (end 113.14 113.6) (width 0.15) (layer F.Cu) (net 2))
   (segment (start 114.2008 121.7581) (end 114.2008 115.0192) (width 0.15) (layer F.Cu) (net 2))
@@
   (segment (start 120.678 102.546) (end 121.6788 103.5468) (width 0.15) (layer F.Cu) (net 2))
   (segment (start 121.6788 103.5468) (end 122.1562 103.5468) (width 0.15) (layer F.Cu) (net 2))
-  (segment (start 122.1562 103.5468) (end 128.1189 109.5095) (width 0.15) (layer F.Cu) (net 2))
-  (segment (start 128.1189 109.5095) (end 128.1189 110.8028) (width 0.15) (layer F.Cu) (net 2))
-  (segment (start 128.1189 110.8028) (end 129.6345 112.3184) (width 0.15) (layer F.Cu) (net 2))
-  (segment (start 129.6345 112.3184) (end 131.7192 112.3184) (width 0.15) (layer F.Cu) (net 2))
-  (segment (start 131.7192 112.3184) (end 137.1678 117.767) (width 0.15) (layer F.Cu) (net 2))
   (segment (start 115.1015 102.594) (end 120.63 102.594) (width 0.15) (layer F.Cu) (net 2))
   (segment (start 120.63 102.594) (end 120.678 102.546) (width 0.15) (layer F.Cu) (net 2))
@@
   (via (at 84.2277 114.325) (size 0.5) (layers F.Cu B.Cu) (net 2))
   (via (at 83.794 110.536) (size 0.5) (layers F.Cu B.Cu) (net 2))
+  (segment (start 115.11 114.7275) (end 116.1025 114.7275) (width 0.15) (layer F.Cu) (net 2))
+  (via (at 118.71876 112.154959) (size 0.5) (drill 0.25) (layers F.Cu B.Cu) (net 2))
+  (segment (start 118.675041 112.154959) (end 118.71876 112.154959) (width 0.15) (layer F.Cu) (net 2))
+  (segment (start 116.1025 114.7275) (end 118.675041 112.154959) (width 0.15) (layer F.Cu) (net 2))
+  (via (at 121.313876 110.236124) (size 0.5) (drill 0.25) (layers F.Cu B.Cu) (net 2))
+  (segment (start 119.646501 111.903499) (end 121.313876 110.236124) (width 0.15) (layer B.Cu) (net 2))
+  (segment (start 119.578001 111.834999) (end 119.646501 111.903499) (width 0.15) (layer B.Cu) (net 2))
+  (segment (start 119.121999 111.834999) (end 119.578001 111.834999) (width 0.15) (layer B.Cu) (net 2))
+  (segment (start 118.874999 112.081999) (end 119.121999 111.834999) (width 0.15) (layer B.Cu) (net 2))
+  (segment (start 118.874999 112.154959) (end 118.874999 112.081999) (width 0.15) (layer B.Cu) (net 2))
+  (segment (start 118.71876 112.154959) (end 118.874999 112.154959) (width 0.15) (layer B.Cu) (net 2))
+  (via (at 122.03 107.71) (size 0.5) (drill 0.25) (layers F.Cu B.Cu) (net 2))
+  (segment (start 122.03 109.52) (end 122.03 107.71) (width 0.15) (layer F.Cu) (net 2))
+  (segment (start 121.313876 110.236124) (end 122.03 109.52) (width 0.15) (layer F.Cu) (net 2))
+  (via (at 124.8397 106.2303) (size 0.5) (drill 0.25) (layers F.Cu B.Cu) (net 2))
+  (segment (start 123.36 107.71) (end 124.8397 106.2303) (width 0.15) (layer B.Cu) (net 2))
+  (segment (start 122.03 107.71) (end 123.36 107.71) (width 0.15) (layer B.Cu) (net 2))
+  (segment (start 122.1562 103.5468) (end 124.8397 106.2303) (width 0.15) (layer F.Cu) (net 2))
   (segment (start 115.1015 104.594) (end 115.1015 104.094) (width 0.15) (layer F.Cu) (net 3))
   (segment (start 116.309 104.578) (end 116.293 104.594) (width 0.15) (layer F.Cu) (net 3))
@@
   (segment (start 114.9102 105.9364) (end 112.2883 103.3145) (width 0.15) (layer B.Cu) (net 3))
   (segment (start 112.2883 103.3145) (end 107.3395 103.3145) (width 0.15) (layer B.Cu) (net 3))
-  (segment (start 115.1326 123.3807) (end 115.1326 106.1588) (width 0.15) (layer B.Cu) (net 3))
+  (segment (start 115.1326 123.3807) (end 115.1326 111.7274) (width 0.15) (layer B.Cu) (net 3))
   (segment (start 115.1326 106.1588) (end 114.9102 105.9364) (width 0.15) (layer B.Cu) (net 3))
   (segment (start 114.9102 105.9364) (end 116.309 104.5376) (width 0.15) (layer B.Cu) (net 3))
@@
   (segment (start 111.7008 128.9492) (end 111.7008 129.8648) (width 0.15) (layer F.Cu) (net 3))
   (segment (start 109.9092 128.9492) (end 109.9 128.94) (width 0.15) (layer F.Cu) (net 3))
+  (segment (start 115.1326 107.6474) (end 115.1326 106.1588) (width 0.15) (layer B.Cu) (net 3))
+  (via (at 115.1326 107.6474) (size 0.5) (drill 0.25) (layers F.Cu B.Cu) (net 3))
+  (segment (start 115.1326 109.8574) (end 115.1326 107.6474) (width 0.15) (layer B.Cu) (net 3))
+  (via (at 115.1326 109.8574) (size 0.5) (drill 0.25) (layers F.Cu B.Cu) (net 3))
+  (segment (start 115.1326 111.7274) (end 115.1326 109.8574) (width 0.15) (layer B.Cu) (net 3))
+  (via (at 115.1326 111.7274) (size 0.5) (drill 0.25) (layers F.Cu B.Cu) (net 3))
   (segment (start 115.11 113.1525) (end 114.414 112.4565) (width 0.15) (layer F.Cu) (net 4))
   (segment (start 114.414 112.4565) (end 114.414 107.2815) (width 0.15) (layer F.Cu) (net 4))
@@
   (segment (start 127.1649 85.764) (end 130.058 85.764) (width 0.15) (layer F.Cu) (net 13))
   (segment (start 127.132 85.764) (end 127.1649 85.764) (width 0.15) (layer F.Cu) (net 13))
-  (segment (start 130.058 85.764) (end 130.058 86.8393) (width 0.15) (layer B.Cu) (net 13))
-  (segment (start 130.058 86.8393) (end 130.192 86.8393) (width 0.15) (layer B.Cu) (net 13))
-  (segment (start 130.192 86.8393) (end 134.903 91.5496) (width 0.15) (layer B.Cu) (net 13))
   (segment (start 124.0661 89.3793) (end 113.414 100.0314) (width 0.15) (layer F.Cu) (net 14))
   (segment (start 113.414 100.0314) (end 113.414 100.4065) (width 0.15) (layer F.Cu) (net 14))
@@
   (segment (start 115.2509 105.2434) (end 115.1015 105.094) (width 0.15) (layer F.Cu) (net 22))
   (segment (start 115.5 105.094) (end 115.6494 105.2434) (width 0.15) (layer F.Cu) (net 22))
-  (segment (start 130.058 121.324) (end 131.133 121.324) (width 0.15) (layer B.Cu) (net 22))
-  (segment (start 131.133 121.324) (end 134.54 117.917) (width 0.15) (layer B.Cu) (net 22))
   (segment (start 115.6064 105.7434) (end 128.593 118.73) (width 0.15) (layer F.Cu) (net 23))
   (segment (start 128.593 118.73) (end 128.593 121.436) (width 0.15) (layer F.Cu) (net 23))
@@
   (segment (start 115.2509 105.7434) (end 115.1015 105.594) (width 0.15) (layer F.Cu) (net 23))
   (segment (start 115.457 105.594) (end 115.6064 105.7434) (width 0.15) (layer F.Cu) (net 23))
-  (segment (start 130.058 123.864) (end 130.058 122.856) (width 0.15) (layer B.Cu) (net 23))
-  (segment (start 130.058 122.856) (end 132.629 120.285) (width 0.15) (layer B.Cu) (net 23))
   (segment (start 122.4005 117.7824) (end 129.947 125.329) (width 0.15) (layer F.Cu) (net 24))
   (segment (start 129.947 125.329) (end 130.058 125.329) (width 0.15) (layer F.Cu) (net 24))

Commit message: ice40qfn restarted: simplest design ready?
Connections:
- net ale renamed rfrx1_false
- net ce renamed rfrx0_false
- net d0 renamed rfrx0_true

Commit message: ice40qfn restarted: simplest design ready?
Connections:
- net re renamed rfrx2_true
- net we renamed rfrx2_false

Commit message: ice40qfn restarted: simplest design ready?
Connections:
- net cle renamed notLVDS
