File: hardware/fpga/ice40std/ice40up5brdV1/ice40up5brdV1/ice40up5.kicad_sch (KiCad schematic)
At the start: 3 parts, among them U1 ICE40UP5K-SG48ITR

Commit message: pwm / lvds power / filters
Connections:
- net +3V3: no longer U1.1 (VCCIO_2), U1.33 (VCCIO_0)
- new net 3V3ANA: U1.33 (VCCIO_0)
- new net 3V3PWM: U1.1 (VCCIO_2)
Changed lines of the file:
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@@
+    )
+  )
+  (global_label "3V3ANA" (shape input) (at 80.01 63.5 90) (fields_autoplaced)
+    (effects (font (size 1.27 1.27)) (justify left))
+    (property "Intersheet References" "${INTERSHEET_REFS}" (id 0) (at 79.9306 54.1606 90)
+      (effects (font (size 1.27 1.27)) (justify left) hide)
     )
   )
@@
     (property "Intersheet References" "${INTERSHEET_REFS}" (id 0) (at 0 0 0)
       (effects (font (size 1.27 1.27)) hide)
+    )
+  )
+  (global_label "3V3PWM" (shape input) (at 189.23 66.04 90) (fields_autoplaced)
+    (effects (font (size 1.27 1.27)) (justify left))
+    (property "Intersheet References" "${INTERSHEET_REFS}" (id 0) (at 189.1506 56.0353 90)
+      (effects (font (size 1.27 1.27)) (justify left) hide)
     )
   )
@@
     (pin "5")
   )
-  (symbol (lib_id "power:+3V3") (at 80.01 63.5 0) (unit 1)
-    (in_bom yes) (on_board yes)
-    (property "Reference" "#PWR01" (id 0) (at 80.01 67.31 0)
-      (effects (font (size 1.27 1.27)) hide)
-    )
-    (property "Value" "+3V3" (id 1) (at 80.391 59.1058 0))
-    (property "Footprint" "" (id 2) (at 80.01 63.5 0)
-      (effects (font (size 1.27 1.27)) hide)
-    )
-    (property "Datasheet" "" (id 3) (at 80.01 63.5 0)
-      (effects (font (size 1.27 1.27)) hide)
-    )
-    (pin "1")
-  )
-  (symbol (lib_id "power:+3V3") (at 189.23 66.04 0) (unit 1)
-    (in_bom yes) (on_board yes)
-    (property "Reference" "#PWR04" (id 0) (at 189.23 69.85 0)
-      (effects (font (size 1.27 1.27)) hide)
-    )
-    (property "Value" "+3V3" (id 1) (at 189.611 61.6458 0))
-    (property "Footprint" "" (id 2) (at 189.23 66.04 0)
-      (effects (font (size 1.27 1.27)) hide)
-    )
-    (property "Datasheet" "" (id 3) (at 189.23 66.04 0)
-      (effects (font (size 1.27 1.27)) hide)
-    )
-    (pin "1")
-  )
   (symbol (lib_id "Device:C") (at 127 49.53 0) (unit 1)

Commit message: pwm / lvds power / filters
Parts:
- added C? (x2): 0.1uF, Capacitor_SMD:C_0402_1005Metric, symbol Device:C
Connections:
- net +3V3 is gone; now on net 3V3ANA: C1.1, C2.1
- net GND: now also C?.2, C?.2
- new net: C?.1, C?.1
Changed lines of the file:
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@@
   (junction (at 134.62 40.64) (diameter 0) (color 0 0 0 0)
+  )
+  (junction (at 243.84 66.0275) (diameter 0) (color 0 0 0 0)
   )
   (no_connect (at 69.85 91.44))
@@
   (no_connect (at 179.07 86.36))
   (no_connect (at 69.85 83.82))
+  (wire (pts (xy 134.62 27.94) (xy 134.62 40.64))
+    (stroke (width 0) (type default) (color 0 0 0 0))
+  )
+  (wire (pts (xy 176.53 88.9) (xy 179.07 88.9))
+    (stroke (width 0) (type default) (color 0 0 0 0))
+  )
+  (wire (pts (xy 243.84 66.0275) (xy 252.73 66.0275))
+    (stroke (width 0) (type default) (color 0 0 0 0))
+  )
+  (wire (pts (xy 252.73 66.0275) (xy 252.73 58.4075))
+    (stroke (width 0) (type default) (color 0 0 0 0))
+  )
+  (wire (pts (xy 127 53.34) (xy 127 60.96))
+    (stroke (width 0) (type default) (color 0 0 0 0))
+  )
+  (wire (pts (xy 127 45.72) (xy 127 40.64))
+    (stroke (width 0) (type default) (color 0 0 0 0))
+  )
+  (wire (pts (xy 80.01 63.5) (xy 80.01 68.58))
+    (stroke (width 0) (type default) (color 0 0 0 0))
+  )
+  (wire (pts (xy 237.49 45.7075) (xy 252.73 45.7075))
+    (stroke (width 0) (type default) (color 0 0 0 0))
+  )
+  (wire (pts (xy 127 60.96) (xy 133.35 60.96))
+    (stroke (width 0) (type default) (color 0 0 0 0))
+  )
+  (wire (pts (xy 237.49 58.4075) (xy 237.49 66.0275))
+    (stroke (width 0) (type default) (color 0 0 0 0))
+  )
+  (wire (pts (xy 176.53 93.98) (xy 179.07 93.98))
+    (stroke (width 0) (type default) (color 0 0 0 0))
+  )
+  (wire (pts (xy 142.24 60.96) (xy 142.24 53.34))
+    (stroke (width 0) (type default) (color 0 0 0 0))
+  )
+  (wire (pts (xy 133.35 60.96) (xy 142.24 60.96))
+    (stroke (width 0) (type default) (color 0 0 0 0))
+  )
+  (wire (pts (xy 252.73 45.7075) (xy 252.73 50.7875))
+    (stroke (width 0) (type default) (color 0 0 0 0))
+  )
+  (wire (pts (xy 237.49 50.7875) (xy 237.49 45.7075))
+    (stroke (width 0) (type default) (color 0 0 0 0))
+  )
+  (wire (pts (xy 237.49 66.0275) (xy 243.84 66.0275))
+    (stroke (width 0) (type default) (color 0 0 0 0))
+  )
+  (wire (pts (xy 243.84 66.0275) (xy 243.84 71.1075))
+    (stroke (width 0) (type default) (color 0 0 0 0))
+  )
+  (wire (pts (xy 133.35 60.96) (xy 133.35 66.04))
+    (stroke (width 0) (type default) (color 0 0 0 0))
+  )
+  (wire (pts (xy 245.11 34.29) (xy 245.11 45.72))
+    (stroke (width 0) (type default) (color 0 0 0 0))
+  )
   (wire (pts (xy 127 40.64) (xy 134.62 40.64))
     (stroke (width 0) (type default) (color 0 0 0 0))
   )
-  (wire (pts (xy 176.53 88.9) (xy 179.07 88.9))
-    (stroke (width 0) (type default) (color 0 0 0 0))
-  )
-  (wire (pts (xy 127 53.34) (xy 127 60.96))
-    (stroke (width 0) (type default) (color 0 0 0 0))
-  )
-  (wire (pts (xy 127 45.72) (xy 127 40.64))
-    (stroke (width 0) (type default) (color 0 0 0 0))
-  )
-  (wire (pts (xy 80.01 63.5) (xy 80.01 68.58))
-    (stroke (width 0) (type default) (color 0 0 0 0))
-  )
-  (wire (pts (xy 127 60.96) (xy 133.35 60.96))
-    (stroke (width 0) (type default) (color 0 0 0 0))
-  )
-  (wire (pts (xy 176.53 93.98) (xy 179.07 93.98))
-    (stroke (width 0) (type default) (color 0 0 0 0))
-  )
-  (wire (pts (xy 142.24 60.96) (xy 142.24 53.34))
-    (stroke (width 0) (type default) (color 0 0 0 0))
-  )
-  (wire (pts (xy 133.35 60.96) (xy 142.24 60.96))
-    (stroke (width 0) (type default) (color 0 0 0 0))
-  )
-  (wire (pts (xy 134.62 34.29) (xy 134.62 40.64))
-    (stroke (width 0) (type default) (color 0 0 0 0))
-  )
-  (wire (pts (xy 133.35 60.96) (xy 133.35 66.04))
+  (wire (pts (xy 142.24 40.64) (xy 142.24 45.72))
+    (stroke (width 0) (type default) (color 0 0 0 0))
+  )
+  (wire (pts (xy 189.23 66.04) (xy 189.23 71.12))
     (stroke (width 0) (type default) (color 0 0 0 0))
   )
   (wire (pts (xy 134.62 40.64) (xy 142.24 40.64))
-    (stroke (width 0) (type default) (color 0 0 0 0))
-  )
-  (wire (pts (xy 142.24 40.64) (xy 142.24 45.72))
-    (stroke (width 0) (type default) (color 0 0 0 0))
-  )
-  (wire (pts (xy 189.23 66.04) (xy 189.23 71.12))
     (stroke (width 0) (type default) (color 0 0 0 0))
   )
@@
     )
   )
+  (global_label "3V3PWM" (shape input) (at 245.11 34.29 90) (fields_autoplaced)
+    (effects (font (size 1.27 1.27)) (justify left))
+    (property "Intersheet References" "${INTERSHEET_REFS}" (id 0) (at 245.0306 24.2853 90)
+      (effects (font (size 1.27 1.27)) (justify left) hide)
+    )
+  )
   (global_label "pwm_o2" (shape input) (at 176.53 93.98 180) (fields_autoplaced)
     (effects (font (size 1.27 1.27)) (justify right))
@@
     (property "Intersheet References" "${INTERSHEET_REFS}" (id 0) (at 166.7068 83.7406 0)
       (effects (font (size 1.27 1.27)) (justify right) hide)
+    )
+  )
+  (global_label "3V3ANA" (shape input) (at 134.62 27.94 90) (fields_autoplaced)
+    (effects (font (size 1.27 1.27)) (justify left))
+    (property "Intersheet References" "${INTERSHEET_REFS}" (id 0) (at 134.5406 18.6006 90)
+      (effects (font (size 1.27 1.27)) (justify left) hide)
     )
   )
@@
     (pin "2")
   )
-  (symbol (lib_id "power:+3V3") (at 134.62 34.29 0) (unit 1)
-    (in_bom yes) (on_board yes)
-    (property "Reference" "#PWR03" (id 0) (at 134.62 38.1 0)
-      (effects (font (size 1.27 1.27)) hide)
-    )
-    (property "Value" "+3V3" (id 1) (at 135.001 29.8958 0))
-    (property "Footprint" "" (id 2) (at 134.62 34.29 0)
-      (effects (font (size 1.27 1.27)) hide)
-    )
-    (property "Datasheet" "" (id 3) (at 134.62 34.29 0)
-      (effects (font (size 1.27 1.27)) hide)
-    )
-    (pin "1")
-  )
   (symbol (lib_id "power:GND") (at 133.35 66.04 0) (unit 1)
     (in_bom yes) (on_board yes)
@@
       (effects (font (size 1.27 1.27)) hide)
     )
+    (pin "1")
+  )
+  (symbol (lib_id "Device:C") (at 237.49 54.5975 0) (unit 1)
+    (in_bom yes) (on_board yes)
+    (property "Reference" "C?" (id 0) (at 240.411 53.4291 0)
+      (effects (font (size 1.27 1.27)) (justify left))
+    )
+    (property "Value" "0.1uF" (id 1) (at 240.411 55.7405 0)
+      (effects (font (size 1.27 1.27)) (justify left))
+    )
+    (property "Footprint" "Capacitor_SMD:C_0402_1005Metric" (id 2) (at 238.4552 58.4075 0)
+      (effects (font (size 1.27 1.27)) hide)
+    )
+    (property "Datasheet" "~" (id 3) (at 237.49 54.5975 0)
+      (effects (font (size 1.27 1.27)) hide)
+    )
+    (pin "1")
+    (pin "2")
+  )
+  (symbol (lib_id "Device:C") (at 252.73 54.5975 0) (unit 1)
+    (in_bom yes) (on_board yes)
+    (property "Reference" "C?" (id 0) (at 255.651 53.4291 0)
+      (effects (font (size 1.27 1.27)) (justify left))
+    )
+    (property "Value" "0.1uF" (id 1) (at 255.651 55.7405 0)
+      (effects (font (size 1.27 1.27)) (justify left))
+    )
+    (property "Footprint" "Capacitor_SMD:C_0402_1005Metric" (id 2) (at 253.6952 58.4075 0)
+      (effects (font (size 1.27 1.27)) hide)
+    )
+    (property "Datasheet" "~" (id 3) (at 252.73 54.5975 0)
+      (effects (font (size 1.27 1.27)) hide)
+    )
+    (pin "1")
+    (pin "2")
+  )
+  (symbol (lib_id "power:GND") (at 243.84 71.1075 0) (unit 1)
+    (in_bom yes) (on_board yes)
+    (property "Reference" "#PWR?" (id 0) (at 243.84 77.4575 0)
+      (effects (font (size 1.27 1.27)) hide)
+    )
+    (property "Value" "GND" (id 1) (at 243.967 75.5017 0))
+    (property "Footprint" "" (id 2) (at 243.84 71.1075 0)
+      (effects (font (size 1.27 1.27)) hide)
+    )
+    (property "Datasheet" "" (id 3) (at 243.84 71.1075 0)
+      (effects (font (size 1.27 1.27)) hide)
+    )

Commit message: pwm / lvds power / filters
Parts:
- gave numbers to parts that had none: 2
Changed lines of the file:
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@@
   (symbol (lib_id "Device:C") (at 237.49 54.5975 0) (unit 1)
     (in_bom yes) (on_board yes)
-    (property "Reference" "C?" (id 0) (at 240.411 53.4291 0)
+    (property "Reference" "C20" (id 0) (at 240.411 53.4291 0)
       (effects (font (size 1.27 1.27)) (justify left))
     )
@@
   (symbol (lib_id "Device:C") (at 252.73 54.5975 0) (unit 1)
     (in_bom yes) (on_board yes)
-    (property "Reference" "C?" (id 0) (at 255.651 53.4291 0)
+    (property "Reference" "C21" (id 0) (at 255.651 53.4291 0)
       (effects (font (size 1.27 1.27)) (justify left))
     )
@@
   (symbol (lib_id "power:GND") (at 243.84 71.1075 0) (unit 1)
     (in_bom yes) (on_board yes)
-    (property "Reference" "#PWR?" (id 0) (at 243.84 77.4575 0)
+    (property "Reference" "#PWR0111" (id 0) (at 243.84 77.4575 0)
       (effects (font (size 1.27 1.27)) hide)
     )

Commit message: pwm / lvds power / filters
Parts:
- C1, C20: value 0.1uF -> 10uF
Changed lines of the file:
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@@
       (effects (font (size 1.27 1.27)) (justify left))
     )
-    (property "Value" "0.1uF" (id 1) (at 129.921 50.673 0)
+    (property "Value" "10uF" (id 1) (at 129.921 50.673 0)
       (effects (font (size 1.27 1.27)) (justify left))
     )
@@
       (effects (font (size 1.27 1.27)) (justify left))
     )
-    (property "Value" "0.1uF" (id 1) (at 240.411 55.7405 0)
+    (property "Value" "10uF" (id 1) (at 240.411 55.7405 0)
       (effects (font (size 1.27 1.27)) (justify left))
     )

Commit message: pwm / lvds power / filters
Parts:
- C1, C20: footprint Capacitor_SMD:C_0402_1005Metric -> Capacitor_SMD:C_1206_3216Metric
Changed lines of the file:
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@@
       (effects (font (size 1.27 1.27)) (justify left))
     )
-    (property "Footprint" "Capacitor_SMD:C_0402_1005Metric" (id 2) (at 127.9652 53.34 0)
+    (property "Footprint" "Capacitor_SMD:C_1206_3216Metric" (id 2) (at 127.9652 53.34 0)
       (effects (font (size 1.27 1.27)) hide)
     )
@@
       (effects (font (size 1.27 1.27)) (justify left))
     )
-    (property "Footprint" "Capacitor_SMD:C_0402_1005Metric" (id 2) (at 238.4552 58.4075 0)
+    (property "Footprint" "Capacitor_SMD:C_1206_3216Metric" (id 2) (at 238.4552 58.4075 0)
       (effects (font (size 1.27 1.27)) hide)
     )

Commit message: pwm / lvds power / filters
Parts:
- C1, C20: footprint Capacitor_SMD:C_1206_3216Metric -> Capacitor_SMD:C_0603_1608Metric
Changed lines of the file:
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@@
       (effects (font (size 1.27 1.27)) (justify left))
     )
-    (property "Footprint" "Capacitor_SMD:C_1206_3216Metric" (id 2) (at 127.9652 53.34 0)
+    (property "Footprint" "Capacitor_SMD:C_0603_1608Metric" (id 2) (at 127.9652 53.34 0)
       (effects (font (size 1.27 1.27)) hide)
     )
@@
       (effects (font (size 1.27 1.27)) (justify left))
     )
-    (property "Footprint" "Capacitor_SMD:C_1206_3216Metric" (id 2) (at 238.4552 58.4075 0)
+    (property "Footprint" "Capacitor_SMD:C_0603_1608Metric" (id 2) (at 238.4552 58.4075 0)
       (effects (font (size 1.27 1.27)) hide)
     )

Commit message: pwm / lvds power / filters
Connections:
- net l2: now also U1.3 (IOB_9b); no longer U1.4 (IOB_8a)
- net l3: now also U1.4 (IOB_8a); no longer U1.3 (IOB_9b)
Changed lines of the file:
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@@
     (stroke (width 0) (type default) (color 0 0 0 0))
   )
-  (global_label "l3" (shape input) (at 179.07 101.6 180) (fields_autoplaced)
+  (global_label "l3" (shape input) (at 179.07 99.06 180) (fields_autoplaced)
     (effects (font (size 1.27 1.27)) (justify right))
-    (property "Intersheet References" "${INTERSHEET_REFS}" (id 0) (at 174.871 101.5206 0)
+    (property "Intersheet References" "${INTERSHEET_REFS}" (id 0) (at 174.871 98.9806 0)
       (effects (font (size 1.27 1.27)) (justify right) hide)
     )
@@
     )
   )
-  (global_label "l2" (shape input) (at 179.07 99.06 180) (fields_autoplaced)
+  (global_label "l2" (shape input) (at 179.07 101.6 180) (fields_autoplaced)
     (effects (font (size 1.27 1.27)) (justify right))
-    (property "Intersheet References" "${INTERSHEET_REFS}" (id 0) (at 174.871 98.9806 0)
+    (property "Intersheet References" "${INTERSHEET_REFS}" (id 0) (at 174.871 101.5206 0)
       (effects (font (size 1.27 1.27)) (justify right) hide)
     )
