File: hardware/analog/basic_lab/labs/simpleLC_pwm/simpleLC/simple_lc.sch (KiCad schematic (older format))
At the start: 6 parts, among them J1 Conn_01x04_Male, J2 Conn_01x02_Male, Q1 FQP27P06

Commit message: PWM => detect / flyback
Parts:
- removed R1: R, Resistor_THT:R_Axial_DIN0207_L6.3mm_D2.5mm_P2.54mm_Vertical, symbol Device:R
- added D?: D, symbol Device:D
Connections:
- wire segments 20 -> 23
Other:
- moved on the sheet: C1, Q1, R2
Changed lines of the file:
@@
 Comment4 ""
 $EndDescr
-Text GLabel 2250 2900 0    50   Input ~ 0
+Text GLabel 2250 3000 0    50   Input ~ 0
 din
 $Comp
 L power:+3.3V #PWR0101
 U 1 1 60C11C18
-P 3250 2000
-F 0 "#PWR0101" H 3250 1850 50  0001 C CNN
-F 1 "+3.3V" H 3265 2173 50  0000 C CNN
-F 2 "" H 3250 2000 50  0001 C CNN
-F 3 "" H 3250 2000 50  0001 C CNN
-	1    3250 2000
+P 1450 1750
+F 0 "#PWR0101" H 1450 1600 50  0001 C CNN
+F 1 "+3.3V" H 1465 1923 50  0000 C CNN
+F 2 "" H 1450 1750 50  0001 C CNN
+F 3 "" H 1450 1750 50  0001 C CNN
+	1    1450 1750
 	1    0    0    -1
 $EndComp
@@
 L power:GND #PWR0102
 U 1 1 60C11E84
-P 3250 3650
-F 0 "#PWR0102" H 3250 3400 50  0001 C CNN
-F 1 "GND" H 3255 3477 50  0000 C CNN
-F 2 "" H 3250 3650 50  0001 C CNN
-F 3 "" H 3250 3650 50  0001 C CNN
-	1    3250 3650
+P 3250 3750
+F 0 "#PWR0102" H 3250 3500 50  0001 C CNN
+F 1 "GND" H 3255 3577 50  0000 C CNN
+F 2 "" H 3250 3750 50  0001 C CNN
+F 3 "" H 3250 3750 50  0001 C CNN
+	1    3250 3750
 	1    0    0    -1
 $EndComp
@@
 L Transistor_FET:FQP27P06 Q1
 U 1 1 60C127AE
-P 3150 2900
-F 0 "Q1" H 3354 2946 50  0000 L CNN
-F 1 "FQP27P06" H 3354 2855 50  0000 L CNN
-F 2 "Package_TO_SOT_THT:TO-220-3_Vertical" H 3350 2825 50  0001 L CIN
-F 3 "https://www.onsemi.com/pub/Collateral/FQP27P06-D.PDF" H 3150 2900 50  0001 L CNN
-	1    3150 2900
-	1    0    0    -1
-$EndComp
-$Comp
-L Device:R R1
-U 1 1 60C12EAB
-P 3250 2300
-F 0 "R1" H 3320 2346 50  0000 L CNN
-F 1 "R" H 3320 2255 50  0000 L CNN
-F 2 "Resistor_THT:R_Axial_DIN0207_L6.3mm_D2.5mm_P2.54mm_Vertical" V 3180 2300 50  0001 C CNN
-F 3 "~" H 3250 2300 50  0001 C CNN
-	1    3250 2300
-	1    0    0    -1
-$EndComp
-Wire Wire Line
-	3250 2000 3250 2150
-Wire Wire Line
-	3250 2450 3250 2550
-Wire Wire Line
-	3250 3100 3250 3200
-Wire Wire Line
-	2250 2900 2950 2900
-Wire Wire Line
-	3250 3500 3250 3650
+P 3150 3000
+F 0 "Q1" H 3354 3046 50  0000 L CNN
+F 1 "FQP27P06" H 3354 2955 50  0000 L CNN
+F 2 "Package_TO_SOT_THT:TO-220-3_Vertical" H 3350 2925 50  0001 L CIN
+F 3 "https://www.onsemi.com/pub/Collateral/FQP27P06-D.PDF" H 3150 3000 50  0001 L CNN
+	1    3150 3000
+	1    0    0    -1
+$EndComp
+Wire Wire Line
+	3250 3200 3250 3300
+Wire Wire Line
+	2250 3000 2950 3000
+Wire Wire Line
+	3250 3600 3250 3750
 $Comp
 L Device:C C1
 U 1 1 60C143B1
-P 5100 2800
-F 0 "C1" H 5215 2846 50  0000 L CNN
-F 1 "C" H 5215 2755 50  0000 L CNN
-F 2 "Capacitor_THT:C_Disc_D3.8mm_W2.6mm_P2.50mm" H 5138 2650 50  0001 C CNN
-F 3 "~" H 5100 2800 50  0001 C CNN
-	1    5100 2800
-	1    0    0    -1
-$EndComp
-Wire Wire Line
-	5100 2550 5100 2650
+P 1450 2500
+F 0 "C1" H 1565 2546 50  0000 L CNN
+F 1 "C" H 1565 2455 50  0000 L CNN
+F 2 "Capacitor_THT:C_Disc_D3.8mm_W2.6mm_P2.50mm" H 1488 2350 50  0001 C CNN
+F 3 "~" H 1450 2500 50  0001 C CNN
+	1    1450 2500
+	1    0    0    -1
+$EndComp
 $Comp
 L power:GND #PWR0104
 U 1 1 60C14856
-P 5100 3150
-F 0 "#PWR0104" H 5100 2900 50  0001 C CNN
-F 1 "GND" H 5105 2977 50  0000 C CNN
-F 2 "" H 5100 3150 50  0001 C CNN
-F 3 "" H 5100 3150 50  0001 C CNN
-	1    5100 3150
-	1    0    0    -1
-$EndComp
-Wire Wire Line
-	5100 2950 5100 3150
+P 1450 2850
+F 0 "#PWR0104" H 1450 2600 50  0001 C CNN
+F 1 "GND" H 1455 2677 50  0000 C CNN
+F 2 "" H 1450 2850 50  0001 C CNN
+F 3 "" H 1450 2850 50  0001 C CNN
+	1    1450 2850
+	1    0    0    -1
+$EndComp
+Wire Wire Line
+	1450 2650 1450 2850
 $Comp
 L Connector:Conn_01x04_Male J1
@@
 L Device:R R2
 U 1 1 60C12C69
-P 3250 3350
-F 0 "R2" H 3320 3396 50  0000 L CNN
-F 1 "R" H 3320 3305 50  0000 L CNN
-F 2 "Resistor_THT:R_Axial_DIN0207_L6.3mm_D2.5mm_P2.54mm_Vertical" V 3180 3350 50  0001 C CNN
-F 3 "~" H 3250 3350 50  0001 C CNN
-	1    3250 3350
-	1    0    0    -1
-$EndComp
-Connection ~ 3250 2550
-Wire Wire Line
-	3250 2550 3250 2700
-Wire Wire Line
-	3250 2550 5100 2550
+P 3250 3450
+F 0 "R2" H 3320 3496 50  0000 L CNN
+F 1 "R" H 3320 3405 50  0000 L CNN
+F 2 "Resistor_THT:R_Axial_DIN0207_L6.3mm_D2.5mm_P2.54mm_Vertical" V 3180 3450 50  0001 C CNN
+F 3 "~" H 3250 3450 50  0001 C CNN
+	1    3250 3450
+	1    0    0    -1
+$EndComp
+Wire Wire Line
+	3250 2650 3250 2750
 $Comp
 L Connector:Conn_01x02_Male J2
@@
 	-1   0    0    1
 $EndComp
-$Comp
-L power:GND #PWR03
-U 1 1 60CA61F3
-P 5750 3150
-F 0 "#PWR03" H 5750 2900 50  0001 C CNN
-F 1 "GND" H 5755 2977 50  0000 C CNN
-F 2 "" H 5750 3150 50  0001 C CNN
-F 3 "" H 5750 3150 50  0001 C CNN
-	1    5750 3150
-	1    0    0    -1
-$EndComp
-Wire Wire Line
-	6150 2650 5750 2650
-Wire Wire Line
-	5750 2650 5750 3150
-Wire Wire Line
-	5100 2550 6150 2550
-Connection ~ 5100 2550
 NoConn ~ 9350 1850
+Wire Wire Line
+	3250 2550 6150 2550
+Wire Wire Line
+	3250 2650 6150 2650
+Wire Wire Line
+	1450 2050 2700 2050
+Wire Wire Line
+	3250 2050 3250 2550
+Wire Wire Line
+	1450 1750 1450 2050
+Wire Wire Line
+	1450 2050 1450 2350
+Connection ~ 1450 2050
+$Comp
+L Device:D D?
+U 1 1 60CD387A
+P 2700 2600
+F 0 "D?" V 2654 2680 50  0000 L CNN
+F 1 "D" V 2745 2680 50  0000 L CNN
+F 2 "" H 2700 2600 50  0001 C CNN
+F 3 "~" H 2700 2600 50  0001 C CNN
+	1    2700 2600
+	0    1    1    0
+$EndComp
+Wire Wire Line
+	2700 2450 2700 2050
+Connection ~ 2700 2050
+Wire Wire Line
+	2700 2050 3250 2050
+Wire Wire Line
+	2700 2750 3250 2750
+Connection ~ 3250 2750
+Wire Wire Line
+	3250 2750 3250 2800
 $EndSCHEMATC

Commit message: PWM => detect / flyback
Parts:
- D1: renamed from D?; footprint (none) -> Diode_THT:D_DO-15_P10.16mm_Horizontal
Changed lines of the file:
@@
 Connection ~ 1450 2050
 $Comp
-L Device:D D?
+L Device:D D1
 U 1 1 60CD387A
 P 2700 2600
-F 0 "D?" V 2654 2680 50  0000 L CNN
+F 0 "D1" V 2654 2680 50  0000 L CNN
 F 1 "D" V 2745 2680 50  0000 L CNN
-F 2 "" H 2700 2600 50  0001 C CNN
+F 2 "Diode_THT:D_DO-15_P10.16mm_Horizontal" H 2700 2600 50  0001 C CNN
 F 3 "~" H 2700 2600 50  0001 C CNN
 	1    2700 2600
