File: hardware/fpga/ice40up5brdV2_only_qfn/ice40up5brdV1/reg.sch (KiCad schematic (older format))
At the start: 16 parts, among them U1 ICE40UP5K-SG48ITR, U2 LTC3406ES5, U3 LTC3406ES5

Commit message: ice40qfn 4layer board started
Parts:
- removed C3, C4: 4.7uF, Capacitor_SMD:C_0402_1005Metric, symbol Device:C
- removed C5, C6: 10uF, Capacitor_SMD:C_0603_1608Metric, symbol Device:C
- removed C7, C8: 0.1uF, Capacitor_SMD:C_0402_1005Metric, symbol Device:C
- removed D1: CDBU0520, Diode_SMD:D_0603_1608Metric, symbol Device:D
- removed L1, L2: L, Inductor_SMD:L_1210_3225Metric, symbol Device:L
- removed R1, R2, R4: 100kOhm, Resistor_SMD:R_0402_1005Metric, symbol Device:R
- removed R3: 450kOhm, Resistor_SMD:R_0402_1005Metric, symbol Device:R
- removed U1: ICE40UP5K-SG48ITR, Package_DFN_QFN:QFN-48-1EP_7x7mm_P0.5mm_EP5.6x5.6mm, symbol FPGA_Lattice:ICE40UP5K-SG48ITR
- removed U2, U3: LTC3406ES5, Package_TO_SOT_SMD:TSOT-23-5, symbol Regulator_Switching:LTC3406ES5
