File: hardware/analog/basic_lab/filters/AFEv4a10Mhz/AFEv4a.kicad_pcb (KiCad board)
At the start: 2 copper layers, 12 parts, among them J1 Connector_Generic_Conn_01x20, J2 Connector_Generic_Conn_01x02

Commit message: ice40qfn restarted: simplest design ready?
Routing:
- net 3V3: track 0.00 -> 8.51 mm
- net Net-(R2-Pad2): track 0.00 -> 3.69 mm
- net rfrx0_false: track 15.4 -> 18.9 mm
- added copper zone on B.Cu, net GND
- added copper zone on F.Cu, net GND
Other:
- board outline added: 49.5 x 55.6 mm
Changed lines of the file:
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@@
   (general
     (thickness 1.6)
-    (drawings 0)
-    (tracks 27)
+    (drawings 4)
+    (tracks 34)
     (zones 0)
     (modules 12)
@@
     )
   )
+  (gr_line (start 148.082 54.61) (end 148.082 109.22) (layer Edge.Cuts) (width 0.1))
+  (gr_line (start 99.314 55.118) (end 148.082 54.61) (layer Edge.Cuts) (width 0.1))
+  (gr_line (start 98.552 110.236) (end 99.314 55.118) (layer Edge.Cuts) (width 0.1))
+  (gr_line (start 148.082 109.22) (end 98.552 110.236) (layer Edge.Cuts) (width 0.1))
   (segment (start 101.54 77.099002) (end 106.05 72.589002) (width 0.25) (layer F.Cu) (net 1))
   (segment (start 101.54 77.9) (end 101.54 77.099002) (width 0.25) (layer F.Cu) (net 1))
@@
   (segment (start 103.886 79.502) (end 104.844999 80.460999) (width 0.25) (layer F.Cu) (net 16))
   (segment (start 104.844999 84.270999) (end 105.918 85.344) (width 0.25) (layer F.Cu) (net 16))
+  (segment (start 105.84 89.09) (end 105.84 85.676) (width 0.25) (layer F.Cu) (net 16))
+  (segment (start 105.84 85.676) (end 105.918 85.598) (width 0.25) (layer F.Cu) (net 16))
+  (segment (start 101.54 57.58) (end 103.554 57.58) (width 0.25) (layer F.Cu) (net 21))
+  (segment (start 103.554 57.58) (end 106.172 60.198) (width 0.25) (layer F.Cu) (net 21))
+  (segment (start 106.172 60.198) (end 106.172 62.992) (width 0.25) (layer F.Cu) (net 21))
   (segment (start 138.989 70.866) (end 143.002 70.866) (width 0.25) (layer F.Cu) (net 22))
   (segment (start 143.002 70.866) (end 143.51 71.374) (width 0.25) (layer F.Cu) (net 22))
+  (segment (start 106.07 76.89) (end 106.07 80.366) (width 0.25) (layer F.Cu) (net 23))
+  (segment (start 106.07 80.366) (end 105.918 80.518) (width 0.25) (layer F.Cu) (net 23))
+  (zone (net 3) (net_name GND) (layer F.Cu) (hatch edge 0.508)
+    (connect_pads (clearance 0.508))
+    (min_thickness 0.254)
+    (fill yes (arc_segments 32) (thermal_gap 0.508) (thermal_bridge_width 0.508))
+    (polygon
+      (pts
+        (xy 164.084 110.998) (xy 91.44 110.49) (xy 92.964 53.594) (xy 163.83 50.8)
+      )
+    )
+  )
+  (zone (net 3) (net_name GND) (layer B.Cu) (hatch edge 0.508)
+    (connect_pads (clearance 0.508))
+    (min_thickness 0.254)
+    (fill yes (arc_segments 32) (thermal_gap 0.508) (thermal_bridge_width 0.508))
+    (polygon
+      (pts
+        (xy 166.37 114.3) (xy 89.662 118.11) (xy 90.17 51.308) (xy 167.132 48.006)
+      )
+    )
+  )
 )

Commit message: ice40qfn restarted: simplest design ready?
Parts:
- added C4: C, Capacitor_THT:C_Axial_L5.1mm_D3.1mm_P15.00mm_Horizontal, F.Cu at (125.7, 63.0)
- added C5: C, Capacitor_THT:C_Axial_L5.1mm_D3.1mm_P15.00mm_Horizontal, F.Cu at (127.3, 88.9)
- added J3: Connector_Generic_Conn_01x02, Connector_PinHeader_2.54mm:PinHeader_1x02_P2.54mm_Vertical, F.Cu at (113.5, 79.0)
Routing:
- net bpf_lvds: track 15.1 -> 24.4 mm
- net rfrx0_false: track 18.9 -> 25.4 mm
- net 3V3: track 8.51 -> 13.2 mm

Commit message: started zero DC-offset AFE
Other:
- net class Default removed
