File: hardware/analog/basic_lab/filters/AFEv4_protoBoard/AFEv4a.kicad_sch (KiCad schematic)
At the start: 17 parts, among them J1 Connector_Generic_Conn_01x20, J2 Connector_Generic_Conn_01x02, J3 Connector_Generic_Conn_01x02, J4 Connector_Generic_Conn_01x02, J5 Connector_Generic_Conn_01x02, J6 Connector_Generic_Conn_01x02

Commit message: started protoboard
Parts:
- removed C1, C2, C3, C4, C5: C, Capacitor_THT:C_Axial_L3.8mm_D2.6mm_P7.50mm_Horizontal, symbol Device:C
- removed J2, J3, J4, J5, J6: Connector_Generic_Conn_01x02, Connector_PinHeader_2.54mm:PinHeader_1x02_P2.54mm_Vertical, symbol bgt:Connector_Generic_Conn_01x02
- removed L1, L2, L3: L, Inductor_THT:L_Toroid_Horizontal_D12.7mm_P20.00mm_Diameter14-5mm_Amidon-T50, symbol Device:L
- removed R1, R2, R4: R, Resistor_THT:R_Axial_DIN0207_L6.3mm_D2.5mm_P5.08mm_Vertical, symbol Device:R
- added J10, J11, J12, J13, J14, J15, J16, J17, J24, J25, J26, J27, J28, J29, J3, J30, J31, J32, J33, J34, J35, J36, J37, J38, J39, J4, J46, J47, J48, J49, J5, J50, J51, J52, J53, J54, J55, J56, J57, J58, J59, J6, J60, J61, J7, J8, J9: Conn_01x06_Male, symbol Connector:Conn_01x06_Male
- added J18: (no value), symbol Connector:Conn_01x12_Male
- added J19, J20, J21, J22, J23, J62: Conn_01x12_Male, symbol Connector:Conn_01x12_Male
- added J2: (no value), symbol Connector:Conn_01x06_Male
- added J40: (no value), symbol Connector:Conn_01x04_Male
- added J41, J42, J43, J44, J45, J63: Conn_01x04_Male, symbol Connector:Conn_01x04_Male
Connections:
- net 3V3: now also J62.1 (Pin_1), J62.10 (Pin_10), J62.11 (Pin_11), J62.12 (Pin_12), J62.2 (Pin_2), J62.3 (Pin_3), J62.4 (Pin_4), J62.5 (Pin_5), J62.6 (Pin_6), J62.7 (Pin_7), J62.8 (Pin_8), J62.9 (Pin_9), J63.1 (Pin_1), J63.2 (Pin_2), J63.3 (Pin_3), J63.4 (Pin_4)
- net GND: now also J18.1 (Pin_1), J18.10 (Pin_10), J18.11 (Pin_11), J18.12 (Pin_12), J18.2 (Pin_2), J18.3 (Pin_3), J18.4 (Pin_4), J18.5 (Pin_5), J18.6 (Pin_6), J18.7 (Pin_7), J18.8 (Pin_8), J18.9 (Pin_9), J19.1 (Pin_1), J19.10 (Pin_10), J19.11 (Pin_11), J19.12 (Pin_12), J19.2 (Pin_2), J19.3 (Pin_3), J19.4 (Pin_4), J19.5 (Pin_5), J19.6 (Pin_6), J19.7 (Pin_7), J19.8 (Pin_8), J19.9 (Pin_9), J20.1 (Pin_1), J20.10 (Pin_10), J20.11 (Pin_11), J20.12 (Pin_12), J20.2 (Pin_2), J20.3 (Pin_3), J20.4 (Pin_4), J20.5 (Pin_5), J20.6 (Pin_6), J20.7 (Pin_7), J20.8 (Pin_8), J20.9 (Pin_9), J21.1 (Pin_1), J21.10 (Pin_10), J21.11 (Pin_11), J21.12 (Pin_12), J21.2 (Pin_2), J21.3 (Pin_3), J21.4 (Pin_4), J21.5 (Pin_5), J21.6 (Pin_6), J21.7 (Pin_7), J21.8 (Pin_8), J21.9 (Pin_9), J22.1 (Pin_1), J22.10 (Pin_10), J22.11 (Pin_11), J22.12 (Pin_12), J22.2 (Pin_2), J22.3 (Pin_3), J22.4 (Pin_4), J22.5 (Pin_5), J22.6 (Pin_6), J22.7 (Pin_7), J22.8 (Pin_8), J22.9 (Pin_9), J23.1 (Pin_1), J23.10 (Pin_10), J23.11 (Pin_11), J23.12 (Pin_12), J23.2 (Pin_2), J23.3 (Pin_3), J23.4 (Pin_4), J23.5 (Pin_5), J23.6 (Pin_6), J23.7 (Pin_7), J23.8 (Pin_8), J23.9 (Pin_9), J40.1 (Pin_1), J40.2 (Pin_2), J40.3 (Pin_3), J40.4 (Pin_4), J41.1 (Pin_1), J41.2 (Pin_2), J41.3 (Pin_3), J41.4 (Pin_4), J42.1 (Pin_1), J42.2 (Pin_2), J42.3 (Pin_3), J42.4 (Pin_4), J43.1 (Pin_1), J43.2 (Pin_2), J43.3 (Pin_3), J43.4 (Pin_4), J44.1 (Pin_1), J44.2 (Pin_2), J44.3 (Pin_3), J44.4 (Pin_4), J45.1 (Pin_1), J45.2 (Pin_2), J45.3 (Pin_3), J45.4 (Pin_4)
- net PWM2: now also J2.1 (Pin_1), J2.2 (Pin_2), J2.3 (Pin_3), J2.4 (Pin_4), J2.5 (Pin_5), J2.6 (Pin_6)
- net pwm_out: now also J3.1 (Pin_1), J3.2 (Pin_2), J3.3 (Pin_3), J3.4 (Pin_4), J3.5 (Pin_5), J3.6 (Pin_6)
- net rfrx0_false: now also J7.1 (Pin_1), J7.2 (Pin_2), J7.3 (Pin_3), J7.4 (Pin_4), J7.5 (Pin_5), J7.6 (Pin_6)
- net rfrx4_false: now reaches J1.10 (Pin_10)
- net rfrx4_false: now also J5.1 (Pin_1), J5.2 (Pin_2), J5.3 (Pin_3), J5.4 (Pin_4), J5.5 (Pin_5), J5.6 (Pin_6)
- net rfrx4_true: now reaches J1.15 (Pin_15)
- net rfrx4_true: now also J4.1 (Pin_1), J4.2 (Pin_2), J4.3 (Pin_3), J4.4 (Pin_4), J4.5 (Pin_5), J4.6 (Pin_6)
- net rfrx2_true: now reaches J1.3 (Pin_3)
- net rfrx2_true: now also J9.1 (Pin_1), J9.2 (Pin_2), J9.3 (Pin_3), J9.4 (Pin_4), J9.5 (Pin_5), J9.6 (Pin_6)
- net rfrx2_false: now reaches J1.4 (Pin_4)
- net rfrx2_false: now also J8.1 (Pin_1), J8.2 (Pin_2), J8.3 (Pin_3), J8.4 (Pin_4), J8.5 (Pin_5), J8.6 (Pin_6)
- net bpf_lvds renamed rfrx0_true
- net rfrx0_true: now also J6.1 (Pin_1), J6.2 (Pin_2), J6.3 (Pin_3), J6.4 (Pin_4), J6.5 (Pin_5), J6.6 (Pin_6)
- new net: J37.1 (Pin_1), J37.2 (Pin_2), J37.3 (Pin_3), J37.4 (Pin_4), J37.5 (Pin_5), J37.6 (Pin_6)
- new net: J35.1 (Pin_1), J35.2 (Pin_2), J35.3 (Pin_3), J35.4 (Pin_4), J35.5 (Pin_5), J35.6 (Pin_6)
- new net: J61.1 (Pin_1), J61.2 (Pin_2), J61.3 (Pin_3), J61.4 (Pin_4), J61.5 (Pin_5), J61.6 (Pin_6)
- new net: J17.1 (Pin_1), J17.2 (Pin_2), J17.3 (Pin_3), J17.4 (Pin_4), J17.5 (Pin_5), J17.6 (Pin_6)
- new net: J47.1 (Pin_1), J47.2 (Pin_2), J47.3 (Pin_3), J47.4 (Pin_4), J47.5 (Pin_5), J47.6 (Pin_6)
- new net: J27.1 (Pin_1), J27.2 (Pin_2), J27.3 (Pin_3), J27.4 (Pin_4), J27.5 (Pin_5), J27.6 (Pin_6)
- new net: J57.1 (Pin_1), J57.2 (Pin_2), J57.3 (Pin_3), J57.4 (Pin_4), J57.5 (Pin_5), J57.6 (Pin_6)
- new net: J38.1 (Pin_1), J38.2 (Pin_2), J38.3 (Pin_3), J38.4 (Pin_4), J38.5 (Pin_5), J38.6 (Pin_6)
- new net: J13.1 (Pin_1), J13.2 (Pin_2), J13.3 (Pin_3), J13.4 (Pin_4), J13.5 (Pin_5), J13.6 (Pin_6)
- new net: J15.1 (Pin_1), J15.2 (Pin_2), J15.3 (Pin_3), J15.4 (Pin_4), J15.5 (Pin_5), J15.6 (Pin_6)
- new net: J26.1 (Pin_1), J26.2 (Pin_2), J26.3 (Pin_3), J26.4 (Pin_4), J26.5 (Pin_5), J26.6 (Pin_6)
- new net: J11.1 (Pin_1), J11.2 (Pin_2), J11.3 (Pin_3), J11.4 (Pin_4), J11.5 (Pin_5), J11.6 (Pin_6)
- new net: J34.1 (Pin_1), J34.2 (Pin_2), J34.3 (Pin_3), J34.4 (Pin_4), J34.5 (Pin_5), J34.6 (Pin_6)
- new net: J16.1 (Pin_1), J16.2 (Pin_2), J16.3 (Pin_3), J16.4 (Pin_4), J16.5 (Pin_5), J16.6 (Pin_6)
- new net: J52.1 (Pin_1), J52.2 (Pin_2), J52.3 (Pin_3), J52.4 (Pin_4), J52.5 (Pin_5), J52.6 (Pin_6)
- new net: J55.1 (Pin_1), J55.2 (Pin_2), J55.3 (Pin_3), J55.4 (Pin_4), J55.5 (Pin_5), J55.6 (Pin_6)
- new net: J49.1 (Pin_1), J49.2 (Pin_2), J49.3 (Pin_3), J49.4 (Pin_4), J49.5 (Pin_5), J49.6 (Pin_6)
- new net: J56.1 (Pin_1), J56.2 (Pin_2), J56.3 (Pin_3), J56.4 (Pin_4), J56.5 (Pin_5), J56.6 (Pin_6)
- new net: J58.1 (Pin_1), J58.2 (Pin_2), J58.3 (Pin_3), J58.4 (Pin_4), J58.5 (Pin_5), J58.6 (Pin_6)
- new net: J28.1 (Pin_1), J28.2 (Pin_2), J28.3 (Pin_3), J28.4 (Pin_4), J28.5 (Pin_5), J28.6 (Pin_6)
- new net: J29.1 (Pin_1), J29.2 (Pin_2), J29.3 (Pin_3), J29.4 (Pin_4), J29.5 (Pin_5), J29.6 (Pin_6)
- new net: J30.1 (Pin_1), J30.2 (Pin_2), J30.3 (Pin_3), J30.4 (Pin_4), J30.5 (Pin_5), J30.6 (Pin_6)
- new net: J53.1 (Pin_1), J53.2 (Pin_2), J53.3 (Pin_3), J53.4 (Pin_4), J53.5 (Pin_5), J53.6 (Pin_6)
- new net: J25.1 (Pin_1), J25.2 (Pin_2), J25.3 (Pin_3), J25.4 (Pin_4), J25.5 (Pin_5), J25.6 (Pin_6)
- new net: J33.1 (Pin_1), J33.2 (Pin_2), J33.3 (Pin_3), J33.4 (Pin_4), J33.5 (Pin_5), J33.6 (Pin_6)
- new net: J60.1 (Pin_1), J60.2 (Pin_2), J60.3 (Pin_3), J60.4 (Pin_4), J60.5 (Pin_5), J60.6 (Pin_6)
- new net: J36.1 (Pin_1), J36.2 (Pin_2), J36.3 (Pin_3), J36.4 (Pin_4), J36.5 (Pin_5), J36.6 (Pin_6)
- new net: J14.1 (Pin_1), J14.2 (Pin_2), J14.3 (Pin_3), J14.4 (Pin_4), J14.5 (Pin_5), J14.6 (Pin_6)
- new net: J51.1 (Pin_1), J51.2 (Pin_2), J51.3 (Pin_3), J51.4 (Pin_4), J51.5 (Pin_5), J51.6 (Pin_6)
- new net: J10.1 (Pin_1), J10.2 (Pin_2), J10.3 (Pin_3), J10.4 (Pin_4), J10.5 (Pin_5), J10.6 (Pin_6)
- new net: J54.1 (Pin_1), J54.2 (Pin_2), J54.3 (Pin_3), J54.4 (Pin_4), J54.5 (Pin_5), J54.6 (Pin_6)
- new net: J46.1 (Pin_1), J46.2 (Pin_2), J46.3 (Pin_3), J46.4 (Pin_4), J46.5 (Pin_5), J46.6 (Pin_6)
- new net: J12.1 (Pin_1), J12.2 (Pin_2), J12.3 (Pin_3), J12.4 (Pin_4), J12.5 (Pin_5), J12.6 (Pin_6)
- new net: J48.1 (Pin_1), J48.2 (Pin_2), J48.3 (Pin_3), J48.4 (Pin_4), J48.5 (Pin_5), J48.6 (Pin_6)
- new net: J59.1 (Pin_1), J59.2 (Pin_2), J59.3 (Pin_3), J59.4 (Pin_4), J59.5 (Pin_5), J59.6 (Pin_6)
- new net: J31.1 (Pin_1), J31.2 (Pin_2), J31.3 (Pin_3), J31.4 (Pin_4), J31.5 (Pin_5), J31.6 (Pin_6)
- new net: J50.1 (Pin_1), J50.2 (Pin_2), J50.3 (Pin_3), J50.4 (Pin_4), J50.5 (Pin_5), J50.6 (Pin_6)
- new net: J39.1 (Pin_1), J39.2 (Pin_2), J39.3 (Pin_3), J39.4 (Pin_4), J39.5 (Pin_5), J39.6 (Pin_6)
- new net: J32.1 (Pin_1), J32.2 (Pin_2), J32.3 (Pin_3), J32.4 (Pin_4), J32.5 (Pin_5), J32.6 (Pin_6)
- new net: J24.1 (Pin_1), J24.2 (Pin_2), J24.3 (Pin_3), J24.4 (Pin_4), J24.5 (Pin_5), J24.6 (Pin_6)
- no-connect marks 9 -> 5

Commit message: started protoboard
Parts:
- J2: value (none) -> Conn_01x06_Male; footprint (none) -> Connector_PinHeader_2.54mm:PinHeader_1x06_P2.54mm_Vertical
Changed lines of the file:
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@@
   (junction (at 134.62 172.72) (diameter 0) (color 0 0 0 0)
   )
+  (junction (at 87.63 97.79) (diameter 0) (color 0 0 0 0)
+  )
   (junction (at 120.65 44.45) (diameter 0) (color 0 0 0 0)
   )
@@
   (junction (at 189.23 146.05) (diameter 0) (color 0 0 0 0)
   )
+  (junction (at 92.71 97.79) (diameter 0) (color 0 0 0 0)
+  )
   (junction (at 96.52 187.96) (diameter 0) (color 0 0 0 0)
   )
@@
   (junction (at 93.98 158.75) (diameter 0) (color 0 0 0 0)
   )
+  (junction (at 97.79 97.79) (diameter 0) (color 0 0 0 0)
+  )
   (junction (at 135.89 44.45) (diameter 0) (color 0 0 0 0)
   )
@@
   (junction (at 166.37 110.49) (diameter 0) (color 0 0 0 0)
   )
-  (junction (at 96.52 97.79) (diameter 0) (color 0 0 0 0)
-  )
   (junction (at 99.06 121.92) (diameter 0) (color 0 0 0 0)
   )
@@
   (junction (at 132.08 187.96) (diameter 0) (color 0 0 0 0)
   )
+  (junction (at 95.25 97.79) (diameter 0) (color 0 0 0 0)
+  )
   (junction (at 194.31 97.79) (diameter 0) (color 0 0 0 0)
   )
@@
   (junction (at 147.32 110.49) (diameter 0) (color 0 0 0 0)
   )
+  (junction (at 90.17 97.79) (diameter 0) (color 0 0 0 0)
+  )
   (junction (at 137.16 97.79) (diameter 0) (color 0 0 0 0)
   )
@@
   (junction (at 189.23 110.49) (diameter 0) (color 0 0 0 0)
   )
-  (junction (at 99.06 97.79) (diameter 0) (color 0 0 0 0)
-  )
-  (junction (at 88.9 97.79) (diameter 0) (color 0 0 0 0)
-  )
   (junction (at 149.86 121.92) (diameter 0) (color 0 0 0 0)
   )
@@
   (junction (at 135.89 76.2) (diameter 0) (color 0 0 0 0)
   )
-  (junction (at 93.98 97.79) (diameter 0) (color 0 0 0 0)
-  )
   (junction (at 109.22 121.92) (diameter 0) (color 0 0 0 0)
   )
@@
   )
   (junction (at 191.77 187.96) (diameter 0) (color 0 0 0 0)
-  )
-  (junction (at 91.44 97.79) (diameter 0) (color 0 0 0 0)
   )
   (junction (at 137.16 121.92) (diameter 0) (color 0 0 0 0)
@@
     (stroke (width 0) (type default) (color 0 0 0 0))
   )
-  (wire (pts (xy 91.44 97.79) (xy 93.98 97.79))
-    (stroke (width 0) (type default) (color 0 0 0 0))
-  )
-  (wire (pts (xy 93.98 97.79) (xy 96.52 97.79))
-    (stroke (width 0) (type default) (color 0 0 0 0))
-  )
   (wire (pts (xy 127 121.92) (xy 129.54 121.92))
     (stroke (width 0) (type default) (color 0 0 0 0))
@@
     (stroke (width 0) (type default) (color 0 0 0 0))
   )
-  (wire (pts (xy 99.06 97.79) (xy 101.6 97.79))
-    (stroke (width 0) (type default) (color 0 0 0 0))
-  )
   (wire (pts (xy 86.36 146.05) (xy 88.9 146.05))
     (stroke (width 0) (type default) (color 0 0 0 0))
@@
     (stroke (width 0) (type default) (color 0 0 0 0))
   )
+  (wire (pts (xy 95.25 97.79) (xy 97.79 97.79))
+    (stroke (width 0) (type default) (color 0 0 0 0))
+  )
   (wire (pts (xy 144.78 187.96) (xy 147.32 187.96))
     (stroke (width 0) (type default) (color 0 0 0 0))
@@
     (stroke (width 0) (type default) (color 0 0 0 0))
   )
+  (wire (pts (xy 87.63 97.79) (xy 90.17 97.79))
+    (stroke (width 0) (type default) (color 0 0 0 0))
+  )
   (wire (pts (xy 152.4 158.75) (xy 154.94 158.75))
     (stroke (width 0) (type default) (color 0 0 0 0))
@@
     (stroke (width 0) (type default) (color 0 0 0 0))
   )
-  (wire (pts (xy 88.9 97.79) (xy 91.44 97.79))
-    (stroke (width 0) (type default) (color 0 0 0 0))
-  )
   (wire (pts (xy 184.15 97.79) (xy 186.69 97.79))
     (stroke (width 0) (type default) (color 0 0 0 0))
@@
     (stroke (width 0) (type default) (color 0 0 0 0))
   )
-  (wire (pts (xy 86.36 97.79) (xy 88.9 97.79))
-    (stroke (width 0) (type default) (color 0 0 0 0))
-  )
   (wire (pts (xy 132.08 187.96) (xy 134.62 187.96))
     (stroke (width 0) (type default) (color 0 0 0 0))
@@
     (stroke (width 0) (type default) (color 0 0 0 0))
   )
+  (wire (pts (xy 90.17 97.79) (xy 92.71 97.79))
+    (stroke (width 0) (type default) (color 0 0 0 0))
+  )
   (wire (pts (xy 242.57 52.07) (xy 245.11 52.07))
     (stroke (width 0) (type default) (color 0 0 0 0))
@@
     (stroke (width 0) (type default) (color 0 0 0 0))
   )
-  (wire (pts (xy 96.52 97.79) (xy 99.06 97.79))
-    (stroke (width 0) (type default) (color 0 0 0 0))
-  )
   (wire (pts (xy 99.06 172.72) (xy 101.6 172.72))
     (stroke (width 0) (type default) (color 0 0 0 0))
@@
     (stroke (width 0) (type default) (color 0 0 0 0))
   )
+  (wire (pts (xy 92.71 97.79) (xy 95.25 97.79))
+    (stroke (width 0) (type default) (color 0 0 0 0))
+  )
   (wire (pts (xy 118.11 67.31) (xy 120.65 67.31))
     (stroke (width 0) (type default) (color 0 0 0 0))
@@
     (stroke (width 0) (type default) (color 0 0 0 0))
   )
+  (wire (pts (xy 97.79 97.79) (xy 100.33 97.79))
+    (stroke (width 0) (type default) (color 0 0 0 0))
+  )
   (wire (pts (xy 148.59 76.2) (xy 151.13 76.2))
     (stroke (width 0) (type default) (color 0 0 0 0))
@@
   )
   (wire (pts (xy 214.63 52.07) (xy 217.17 52.07))
+    (stroke (width 0) (type default) (color 0 0 0 0))
+  )
+  (wire (pts (xy 86.36 97.79) (xy 87.63 97.79))
     (stroke (width 0) (type default) (color 0 0 0 0))
   )
@@
     (pin "6")
   )
-  (symbol (lib_id "Connector:Conn_01x06_Male") (at 96.52 92.71 270) (unit 1)
-    (in_bom yes) (on_board yes) (fields_autoplaced)
-    (property "Reference" "J2" (id 0) (at 95.25 89.061 90))
-    (property "Value" "" (id 1) (at 95.25 91.5979 90))
-    (property "Footprint" "" (id 2) (at 96.52 92.71 0)
-      (effects (font (size 1.27 1.27)) hide)
-    )
-    (property "Datasheet" "~" (id 3) (at 96.52 92.71 0)
-      (effects (font (size 1.27 1.27)) hide)
-    )
-    (pin "1")
-    (pin "2")
-    (pin "3")
-    (pin "4")
-    (pin "5")
-    (pin "6")
-  )
   (symbol (lib_id "Connector:Conn_01x06_Male") (at 191.77 182.88 270) (unit 1)
     (in_bom yes) (on_board yes) (fields_autoplaced)
@@
     (pin "6")
   )
+  (symbol (lib_id "Connector:Conn_01x06_Male") (at 95.25 92.71 270) (unit 1)
+    (in_bom yes) (on_board yes) (fields_autoplaced)
+    (property "Reference" "J2" (id 0) (at 93.98 89.061 90))
+    (property "Value" "Conn_01x06_Male" (id 1) (at 93.98 91.5979 90))
+    (property "Footprint" "Connector_PinHeader_2.54mm:PinHeader_1x06_P2.54mm_Vertical" (id 2) (at 95.25 92.71 0)
+      (effects (font (size 1.27 1.27)) hide)
+    )
+    (property "Datasheet" "~" (id 3) (at 95.25 92.71 0)
+      (effects (font (size 1.27 1.27)) hide)
+    )
+    (pin "1")
+    (pin "2")
+    (pin "3")
+    (pin "4")
+    (pin "5")
+    (pin "6")
+  )
   (symbol (lib_id "Connector:Conn_01x06_Male") (at 114.3 140.97 270) (unit 1)
     (in_bom yes) (on_board yes) (fields_autoplaced)
@@
       (reference "J1") (unit 1) (value "Connector_Generic_Conn_01x20") (footprint "Connector_PinHeader_2.54mm:PinHeader_1x20_P2.54mm_Vertical")
     )
-    (path "/0f87f1f3-0445-434a-bdcc-6b1162948ef1"
-      (reference "J2") (unit 1) (value "Conn_01x06_Male") (footprint "")
+    (path "/b3642838-c802-420a-a759-2110779b0f1c"
+      (reference "J2") (unit 1) (value "Conn_01x06_Male") (footprint "Connector_PinHeader_2.54mm:PinHeader_1x06_P2.54mm_Vertical")
     )
     (path "/a2bfca6c-89bf-4dd1-b627-5c21e60d8fc9"
