File: hardware/analog/basic_lab/analog_labs/AFEv4_attenuator/AFEv4a.kicad_sch (KiCad schematic)
At the start: 63 parts, among them J1 Connector_Generic_Conn_01x20, J10 Conn_01x06_Male, J11 Conn_01x06_Male, J12 Conn_01x06_Male, J13 Conn_01x06_Male, J14 Conn_01x06_Male, J15 Conn_01x06_Male, J16 Conn_01x06_Male, J17 Conn_01x06_Male, J19 Conn_01x12_Male, J2 Conn_01x06_Male, J20 Conn_01x12_Male, J21 Conn_01x12_Male, J22 Conn_01x12_Male, J23 Conn_01x12_Male, J24 Conn_01x06_Male, J25 Conn_01x06_Male, J26 Conn_01x06_Male, J27 Conn_01x06_Male, J28 Conn_01x06_Male, J29 Conn_01x06_Male, J3 Conn_01x06_Male, J30 Conn_01x06_Male, J31 Conn_01x06_Male, J32 Conn_01x06_Male, J33 Conn_01x06_Male, J34 Conn_01x06_Male, J35 Conn_01x06_Male, J36 Conn_01x06_Male, J37 Conn_01x06_Male, J38 Conn_01x06_Male, J39 Conn_01x06_Male, J4 Conn_01x06_Male, J41 Conn_01x04_Male, J42 Conn_01x04_Male, J43 Conn_01x04_Male, J44 Conn_01x04_Male, J45 Conn_01x04_Male, J46 Conn_01x06_Male, J47 Conn_01x06_Male, J48 Conn_01x06_Male, J49 Conn_01x06_Male, J5 Conn_01x06_Male, J50 Conn_01x06_Male, J51 Conn_01x06_Male, J52 Conn_01x06_Male, J53 Conn_01x06_Male, J54 Conn_01x06_Male, J55 Conn_01x06_Male, J56 Conn_01x06_Male, J57 Conn_01x06_Male, J58 Conn_01x06_Male, J59 Conn_01x06_Male, J6 Conn_01x06_Male, J60 Conn_01x06_Male, J61 Conn_01x06_Male, J62 Conn_01x12_Male, J63 Conn_01x04_Male, J7 Conn_01x06_Male, J8 Conn_01x06_Male, J9 Conn_01x06_Male

Commit message: started analog labs
Parts:
- removed J10, J11, J12, J13, J14, J15, J16, J17, J24, J25, J26, J27, J28, J29, J3, J30, J31, J32, J33, J34, J35, J36, J37, J38, J39, J4, J46, J47, J48, J49, J5, J50, J51, J52, J53, J54, J55, J56, J57, J58, J59, J6, J60, J61, J7, J8, J9: Conn_01x06_Male, symbol Connector:Conn_01x06_Male
- removed J18: (no value), symbol Connector:Conn_01x12_Male
- removed J19, J20, J21, J22, J23, J62: Conn_01x12_Male, symbol Connector:Conn_01x12_Male
- removed J2: Conn_01x06_Male, Connector_PinHeader_2.54mm:PinHeader_1x06_P2.54mm_Vertical, symbol Connector:Conn_01x06_Male
- removed J40: (no value), symbol Connector:Conn_01x04_Male
- removed J41, J42, J43, J44, J45, J63: Conn_01x04_Male, symbol Connector:Conn_01x04_Male

Commit message: started analog labs
Parts:
- added C?: (no value), symbol Device:C
- added R? (x3): (no value), symbol Device:R
Connections:
- net 3V3: now also R?.1
- net GND: now also C?.2, R?.2
- net pwm_out: now also R?.1
- net rfrx0_false: now also C?.1, R?.2
- net rfrx0_true renamed atten_in
- net atten_in: now also R?.1, R?.2
- net rfrx2_false: no longer names the net of J1.4 (Pin_4)
- net rfrx2_true: no longer names the net of J1.3 (Pin_3)
- net rfrx4_false: no longer names the net of J1.10 (Pin_10)
- net rfrx4_true: no longer names the net of J1.15 (Pin_15)
- no-connect marks 5 -> 9

Commit message: started analog labs
Parts:
- added R1, R2, R3, R4, R5, R7, R8, R9: (no value), symbol Device:R
- gave numbers to parts that had none: 4
Connections:
- net 3V3: now also R1.1, R4.1, R8.1
- net GND: now also R2.2, R5.2, R9.2
- net PWM2: now also R7.2, R8.2, R9.1
- net atten_in: now also R1.2, R2.1, R3.1
- new net: R3.2, R4.2, R5.1, R7.1

Commit message: started analog labs
Parts:
- removed R2: (no value), symbol Device:R
- R1: value (none) -> R
Connections:
- net 3V3: no longer R1.1
- net PWM2: now also R1.2; no longer R7.2, R8.2, R9.1
- net atten_in: no longer R1.2
- new net: R1.1, R7.2, R8.2, R9.1
Changed lines of the file:
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@@
 (kicad_sch (version 20211123) (generator eeschema)
   (paper "A4")
-  (junction (at 127 142.24) (diameter 0) (color 0 0 0 0)
-  )
   (junction (at 140.97 100.33) (diameter 0) (color 0 0 0 0)
   )
   (junction (at 140.97 142.24) (diameter 0) (color 0 0 0 0)
-  )
-  (junction (at 127 100.33) (diameter 0) (color 0 0 0 0)
-  )
-  (junction (at 127 120.65) (diameter 0) (color 0 0 0 0)
   )
   (junction (at 140.97 120.65) (diameter 0) (color 0 0 0 0)
@@
     (stroke (width 0) (type default) (color 0 0 0 0))
   )
-  (wire (pts (xy 119.38 120.65) (xy 127 120.65))
-    (stroke (width 0) (type default) (color 0 0 0 0))
-  )
-  (wire (pts (xy 127 100.33) (xy 127 106.68))
-    (stroke (width 0) (type default) (color 0 0 0 0))
-  )
   (wire (pts (xy 162.56 120.65) (xy 162.56 128.27))
     (stroke (width 0) (type default) (color 0 0 0 0))
   )
-  (wire (pts (xy 116.84 100.33) (xy 127 100.33))
-    (stroke (width 0) (type default) (color 0 0 0 0))
-  )
   (wire (pts (xy 140.97 100.33) (xy 140.97 106.68))
     (stroke (width 0) (type default) (color 0 0 0 0))
@@
     (stroke (width 0) (type default) (color 0 0 0 0))
   )
-  (wire (pts (xy 162.56 120.65) (xy 167.64 120.65))
+  (wire (pts (xy 162.56 120.65) (xy 177.8 120.65))
     (stroke (width 0) (type default) (color 0 0 0 0))
   )
@@
     (stroke (width 0) (type default) (color 0 0 0 0))
   )
-  (wire (pts (xy 127 120.65) (xy 127 128.27))
-    (stroke (width 0) (type default) (color 0 0 0 0))
-  )
   (wire (pts (xy 140.97 114.3) (xy 140.97 120.65))
     (stroke (width 0) (type default) (color 0 0 0 0))
   )
-  (wire (pts (xy 116.84 142.24) (xy 127 142.24))
+  (wire (pts (xy 185.42 120.65) (xy 198.12 120.65))
     (stroke (width 0) (type default) (color 0 0 0 0))
   )
@@
     (stroke (width 0) (type default) (color 0 0 0 0))
   )
-  (wire (pts (xy 127 120.65) (xy 130.81 120.65))
+  (wire (pts (xy 119.38 120.65) (xy 130.81 120.65))
     (stroke (width 0) (type default) (color 0 0 0 0))
   )
@@
     (stroke (width 0) (type default) (color 0 0 0 0))
   )
-  (wire (pts (xy 127 100.33) (xy 140.97 100.33))
+  (wire (pts (xy 116.84 100.33) (xy 140.97 100.33))
     (stroke (width 0) (type default) (color 0 0 0 0))
   )
@@
     (stroke (width 0) (type default) (color 0 0 0 0))
   )
-  (wire (pts (xy 127 135.89) (xy 127 142.24))
-    (stroke (width 0) (type default) (color 0 0 0 0))
-  )
   (wire (pts (xy 186.69 50.8) (xy 186.69 54.61))
     (stroke (width 0) (type default) (color 0 0 0 0))
@@
     (stroke (width 0) (type default) (color 0 0 0 0))
   )
-  (wire (pts (xy 127 114.3) (xy 127 120.65))
-    (stroke (width 0) (type default) (color 0 0 0 0))
-  )
-  (wire (pts (xy 127 142.24) (xy 140.97 142.24))
+  (wire (pts (xy 116.84 142.24) (xy 140.97 142.24))
     (stroke (width 0) (type default) (color 0 0 0 0))
   )
@@
     )
   )
-  (global_label "PWM2" (shape input) (at 167.64 120.65 0) (fields_autoplaced)
-    (effects (font (size 1.27 1.27)) (justify left))
-    (property "Intersheet References" "${INTERSHEET_REFS}" (id 0) (at 175.3466 120.5706 0)
+  (global_label "PWM2" (shape input) (at 198.12 120.65 0) (fields_autoplaced)
+    (effects (font (size 1.27 1.27)) (justify left))
+    (property "Intersheet References" "${INTERSHEET_REFS}" (id 0) (at 205.8266 120.5706 0)
       (effects (font (size 1.27 1.27)) (justify left) hide)
     )
@@
     (pin "2")
   )
-  (symbol (lib_id "Device:R") (at 127 132.08 0) (unit 1)
-    (in_bom yes) (on_board yes) (fields_autoplaced)
-    (property "Reference" "R2" (id 0) (at 128.778 131.2453 0)
-      (effects (font (size 1.27 1.27)) (justify left))
-    )
-    (property "Value" "" (id 1) (at 128.778 133.7822 0)
-      (effects (font (size 1.27 1.27)) (justify left))
-    )
-    (property "Footprint" "" (id 2) (at 125.222 132.08 90)
-      (effects (font (size 1.27 1.27)) hide)
-    )
-    (property "Datasheet" "~" (id 3) (at 127 132.08 0)
-      (effects (font (size 1.27 1.27)) hide)
-    )
-    (pin "1")
-    (pin "2")
-  )
   (symbol (lib_id "Device:R") (at 162.56 132.08 0) (unit 1)
     (in_bom yes) (on_board yes) (fields_autoplaced)
@@
     )
     (property "Datasheet" "~" (id 3) (at 162.56 132.08 0)
-      (effects (font (size 1.27 1.27)) hide)
-    )
-    (pin "1")
-    (pin "2")
-  )
-  (symbol (lib_id "Device:R") (at 127 110.49 0) (unit 1)
-    (in_bom yes) (on_board yes) (fields_autoplaced)
-    (property "Reference" "R1" (id 0) (at 128.778 109.6553 0)
-      (effects (font (size 1.27 1.27)) (justify left))
-    )
-    (property "Value" "" (id 1) (at 128.778 112.1922 0)
-      (effects (font (size 1.27 1.27)) (justify left))
-    )
-    (property "Footprint" "" (id 2) (at 125.222 110.49 90)
-      (effects (font (size 1.27 1.27)) hide)
-    )
-    (property "Datasheet" "~" (id 3) (at 127 110.49 0)
       (effects (font (size 1.27 1.27)) hide)
     )
@@
     (pin "2")
   )
+  (symbol (lib_id "Device:R") (at 181.61 120.65 90) (unit 1)
+    (in_bom yes) (on_board yes) (fields_autoplaced)
+    (property "Reference" "R1" (id 0) (at 181.61 115.9342 90))
+    (property "Value" "R" (id 1) (at 181.61 118.4711 90))
+    (property "Footprint" "" (id 2) (at 181.61 122.428 90)
+      (effects (font (size 1.27 1.27)) hide)
+    )
+    (property "Datasheet" "~" (id 3) (at 181.61 120.65 0)
+      (effects (font (size 1.27 1.27)) hide)
+    )
+    (pin "1")
+    (pin "2")
+  )
   (symbol (lib_id "Device:R") (at 146.05 62.23 0) (unit 1)
     (in_bom yes) (on_board yes) (fields_autoplaced)
@@
       (reference "J1") (unit 1) (value "Connector_Generic_Conn_01x20") (footprint "Connector_PinHeader_2.54mm:PinHeader_1x20_P2.54mm_Vertical")
     )
-    (path "/1d16b0f9-6d69-4cf5-b1d5-a61070a12b57"
+    (path "/7094677d-5dd7-427a-b179-e2529252d057"
       (reference "R1") (unit 1) (value "R") (footprint "")
     )
-    (path "/1169c561-e31f-4efa-9a6d-0cf86ada0778"
-      (reference "R2") (unit 1) (value "R") (footprint "")
-    )
     (path "/2061f02d-bf2d-4cf0-838d-e927d32e6cd2"

Commit message: started analog labs
Parts:
- added C2: C, Capacitor_THT:C_Axial_L3.8mm_D2.6mm_P7.50mm_Horizontal, symbol Device:C
Connections:
- net 3V3: now also C2.1
- net GND: now also C2.2
Changed lines of the file:
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@@
+    (stroke (width 0) (type default) (color 0 0 0 0))
+  )
+  (wire (pts (xy 240.03 58.42) (xy 255.27 58.42))
     (stroke (width 0) (type default) (color 0 0 0 0))
   )
@@
     (stroke (width 0) (type default) (color 0 0 0 0))
   )
+  (wire (pts (xy 255.27 77.47) (xy 255.27 73.66))
+    (stroke (width 0) (type default) (color 0 0 0 0))
+  )
   (wire (pts (xy 146.05 69.85) (xy 146.05 76.2))
     (stroke (width 0) (type default) (color 0 0 0 0))
@@
     (stroke (width 0) (type default) (color 0 0 0 0))
   )
+  (wire (pts (xy 255.27 58.42) (xy 255.27 66.04))
+    (stroke (width 0) (type default) (color 0 0 0 0))
+  )
   (wire (pts (xy 162.56 114.3) (xy 162.56 120.65))
+    (stroke (width 0) (type default) (color 0 0 0 0))
+  )
+  (wire (pts (xy 240.03 77.47) (xy 255.27 77.47))
     (stroke (width 0) (type default) (color 0 0 0 0))
   )
@@
     )
   )
+  (global_label "3V3" (shape input) (at 240.03 58.42 180) (fields_autoplaced)
+    (effects (font (size 1.27 1.27)) (justify right))
+    (property "Intersheet References" "${INTERSHEET_REFS}" (id 0) (at 285.75 163.83 0)
+      (effects (font (size 1.27 1.27)) hide)
+    )
+  )
   (global_label "GND" (shape input) (at 45.72 80.01 0) (fields_autoplaced)
     (effects (font (size 1.27 1.27)) (justify left))
@@
     (effects (font (size 1.27 1.27)) (justify left))
     (property "Intersheet References" "${INTERSHEET_REFS}" (id 0) (at 0 0 0)
+      (effects (font (size 1.27 1.27)) hide)
+    )
+  )
+  (global_label "GND" (shape input) (at 240.03 77.47 180) (fields_autoplaced)
+    (effects (font (size 1.27 1.27)) (justify right))
+    (property "Intersheet References" "${INTERSHEET_REFS}" (id 0) (at 285.75 170.18 0)
       (effects (font (size 1.27 1.27)) hide)
     )
@@
     (pin "2")
   )
+  (symbol (lib_id "Device:C") (at 255.27 69.85 0) (unit 1)
+    (in_bom yes) (on_board yes) (fields_autoplaced)
+    (property "Reference" "C2" (id 0) (at 258.191 69.0153 0)
+      (effects (font (size 1.27 1.27)) (justify left))
+    )
+    (property "Value" "C" (id 1) (at 258.191 71.5522 0)
+      (effects (font (size 1.27 1.27)) (justify left))
+    )
+    (property "Footprint" "Capacitor_THT:C_Axial_L3.8mm_D2.6mm_P7.50mm_Horizontal" (id 2) (at 256.2352 73.66 0)
+      (effects (font (size 1.27 1.27)) hide)
+    )
+    (property "Datasheet" "~" (id 3) (at 255.27 69.85 0)
+      (effects (font (size 1.27 1.27)) hide)
+    )
+    (pin "1")
+    (pin "2")
+  )
   (symbol (lib_id "Device:R") (at 186.69 58.42 0) (unit 1)
     (in_bom yes) (on_board yes) (fields_autoplaced)
@@
   (symbol_instances
     (path "/21d157b2-f423-42e7-b693-fe99fd35023e"
-      (reference "C1") (unit 1) (value "C") (footprint "")
+      (reference "C1") (unit 1) (value "C") (footprint "Capacitor_THT:C_Axial_L3.8mm_D2.6mm_P7.50mm_Horizontal")
+    )
+    (path "/34c0221c-dfd6-4693-83c9-89363b0d1933"
+      (reference "C2") (unit 1) (value "C") (footprint "Capacitor_THT:C_Axial_L3.8mm_D2.6mm_P7.50mm_Horizontal")
     )
     (path "/00000000-0000-0000-0000-000061f5f9b7"
@@
     )
     (path "/7094677d-5dd7-427a-b179-e2529252d057"
-      (reference "R1") (unit 1) (value "R") (footprint "")
+      (reference "R1") (unit 1) (value "R") (footprint "Connector_PinSocket_2.54mm:PinSocket_1x02_P2.54mm_Vertical")
     )
     (path "/2061f02d-bf2d-4cf0-838d-e927d32e6cd2"
-      (reference "R3") (unit 1) (value "R") (footprint "")
+      (reference "R3") (unit 1) (value "R") (footprint "Connector_PinSocket_2.54mm:PinSocket_1x02_P2.54mm_Vertical")
     )
     (path "/51831213-524b-48d3-aebd-7adee0bbfc5d"
-      (reference "R4") (unit 1) (value "R") (footprint "")
+      (reference "R4") (unit 1) (value "R") (footprint "Resistor_THT:R_Axial_DIN0309_L9.0mm_D3.2mm_P12.70mm_Horizontal")
     )
     (path "/ff470d1b-4094-473e-982b-652022f09e2f"
-      (reference "R5") (unit 1) (value "R") (footprint "")
+      (reference "R5") (unit 1) (value "R") (footprint "Resistor_THT:R_Axial_DIN0309_L9.0mm_D3.2mm_P12.70mm_Horizontal")
     )
     (path "/775b4a34-9736-4b65-bf61-c6c659dab920"
-      (reference "R6") (unit 1) (value "R") (footprint "")
+      (reference "R6") (unit 1) (value "R") (footprint "Resistor_THT:R_Axial_DIN0309_L9.0mm_D3.2mm_P12.70mm_Horizontal")
     )
     (path "/57882615-c6ce-49f0-a554-5c7ea2a1d560"
-      (reference "R7") (unit 1) (value "R") (footprint "")
+      (reference "R7") (unit 1) (value "R") (footprint "Connector_PinSocket_2.54mm:PinSocket_1x02_P2.54mm_Vertical")
     )
     (path "/065fd7cf-e3d4-41f2-8782-2f0ddf9246df"
-      (reference "R8") (unit 1) (value "R") (footprint "")
+      (reference "R8") (unit 1) (value "R") (footprint "Resistor_THT:R_Axial_DIN0309_L9.0mm_D3.2mm_P12.70mm_Horizontal")
     )
     (path "/132bf5df-7d4d-4ba3-9b45-410d2080b9a1"
-      (reference "R9") (unit 1) (value "R") (footprint "")
+      (reference "R9") (unit 1) (value "R") (footprint "Resistor_THT:R_Axial_DIN0309_L9.0mm_D3.2mm_P12.70mm_Horizontal")
     )
     (path "/45e7789e-c256-4f26-8c2f-c77bcf5a6eef"
-      (reference "R10") (unit 1) (value "R") (footprint "")
+      (reference "R10") (unit 1) (value "R") (footprint "Resistor_THT:R_Axial_DIN0309_L9.0mm_D3.2mm_P12.70mm_Horizontal")
     )
     (path "/0a32cbce-6479-432a-a803-9704bd17dde9"
-      (reference "R11") (unit 1) (value "R") (footprint "")
-    )
-  )
+      (reference "R11") (unit 1) (value "R") (footprint "Resistor_THT:R_Axial_DIN0309_L9.0mm_D3.2mm_P12.70mm_Horizontal")
+    )
+  )
