File: hardware/analog/basic_lab/filters/AFEv4_bc847_amp/connector.kicad_sch (KiCad schematic)
At the start: 3 parts, among them J1 Connector_Generic_Conn_01x20

Commit message: started PCB LC LPF
Parts:
- removed C1: C, Capacitor_SMD:C_1206_3216Metric, symbol Device:C
- removed J1: Connector_Generic_Conn_01x20, Connector_PinHeader_2.54mm:PinHeader_1x20_P2.54mm_Vertical, symbol bgt:Connector_Generic_Conn_01x20
- removed R9: R, Resistor_SMD:R_0805_2012Metric, symbol Device:R
Connections:
- no-connect marks 6 -> 0
Changed lines of the file:
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@@
 (kicad_sch (version 20211123) (generator eeschema)
   (paper "A4")
-  (no_connect (at 59.69 77.47))
-  (no_connect (at 59.69 54.61))
-  (no_connect (at 59.69 72.39))
-  (no_connect (at 59.69 90.17))
-  (no_connect (at 59.69 57.15))
-  (no_connect (at 59.69 64.77))
-  (wire (pts (xy 140.97 116.84) (xy 140.97 128.27))
-    (stroke (width 0) (type default) (color 0 0 0 0))
-  )
-  (wire (pts (xy 140.97 116.84) (xy 151.13 116.84))
-    (stroke (width 0) (type default) (color 0 0 0 0))
-  )
-  (wire (pts (xy 154.94 74.93) (xy 154.94 72.39))
-    (stroke (width 0) (type default) (color 0 0 0 0))
-  )
-  (wire (pts (xy 127 97.79) (xy 133.35 97.79))
-    (stroke (width 0) (type default) (color 0 0 0 0))
-  )
-  (wire (pts (xy 111.76 97.79) (xy 119.38 97.79))
-    (stroke (width 0) (type default) (color 0 0 0 0))
-  )
-  (wire (pts (xy 154.94 64.77) (xy 154.94 63.5))
-    (stroke (width 0) (type default) (color 0 0 0 0))
-  )
-  (global_label "GND" (shape input) (at 154.94 63.5 90) (fields_autoplaced)
-    (effects (font (size 1.27 1.27)) (justify left))
-    (property "Intersheet References" "${INTERSHEET_REFS}" (id 0) (at 85.09 149.86 0)
-      (effects (font (size 1.27 1.27)) hide)
-    )
-  )
-  (global_label "rfrx1_false" (shape input) (at 59.69 92.71 0) (fields_autoplaced)
-    (effects (font (size 1.27 1.27)) (justify left))
-    (property "Intersheet References" "${INTERSHEET_REFS}" (id 0) (at 72.1742 92.6306 0)
-      (effects (font (size 1.27 1.27)) (justify left) hide)
-    )
-  )
-  (global_label "GND" (shape input) (at 59.69 82.55 0) (fields_autoplaced)
-    (effects (font (size 1.27 1.27)) (justify left))
-    (property "Intersheet References" "${INTERSHEET_REFS}" (id 0) (at 13.97 -5.08 0)
-      (effects (font (size 1.27 1.27)) hide)
-    )
-  )
-  (global_label "rfrx0_false" (shape input) (at 59.69 85.09 0) (fields_autoplaced)
-    (effects (font (size 1.27 1.27)) (justify left))
-    (property "Intersheet References" "${INTERSHEET_REFS}" (id 0) (at 13.97 -5.08 0)
-      (effects (font (size 1.27 1.27)) hide)
-    )
-  )
-  (global_label "rfrx0_pwm" (shape input) (at 59.69 69.85 0) (fields_autoplaced)
-    (effects (font (size 1.27 1.27)) (justify left))
-    (property "Intersheet References" "${INTERSHEET_REFS}" (id 0) (at 71.6904 69.7706 0)
-      (effects (font (size 1.27 1.27)) (justify left) hide)
-    )
-  )
-  (global_label "rfrx0_true" (shape input) (at 59.69 80.01 0) (fields_autoplaced)
-    (effects (font (size 1.27 1.27)) (justify left))
-    (property "Intersheet References" "${INTERSHEET_REFS}" (id 0) (at 13.97 -5.08 0)
-      (effects (font (size 1.27 1.27)) hide)
-    )
-  )
-  (global_label "GND" (shape input) (at 59.69 52.07 0) (fields_autoplaced)
-    (effects (font (size 1.27 1.27)) (justify left))
-    (property "Intersheet References" "${INTERSHEET_REFS}" (id 0) (at 13.97 -27.94 0)
-      (effects (font (size 1.27 1.27)) hide)
-    )
-  )
-  (global_label "rfrx1_pwm" (shape input) (at 59.69 97.79 0) (fields_autoplaced)
-    (effects (font (size 1.27 1.27)) (justify left))
-    (property "Intersheet References" "${INTERSHEET_REFS}" (id 0) (at 71.6904 97.7106 0)
-      (effects (font (size 1.27 1.27)) (justify left) hide)
-    )
-  )
-  (global_label "3V3" (shape input) (at 133.35 97.79 0) (fields_autoplaced)
-    (effects (font (size 1.27 1.27)) (justify left))
-    (property "Intersheet References" "${INTERSHEET_REFS}" (id 0) (at 87.63 -7.62 0)
-      (effects (font (size 1.27 1.27)) hide)
-    )
-  )
-  (global_label "PWR" (shape input) (at 111.76 97.79 180) (fields_autoplaced)
-    (effects (font (size 1.27 1.27)) (justify right))
-    (property "Intersheet References" "${INTERSHEET_REFS}" (id 0) (at 105.4444 97.7106 0)
-      (effects (font (size 1.27 1.27)) (justify right) hide)
-    )
-  )
-  (global_label "GND" (shape input) (at 59.69 59.69 0) (fields_autoplaced)
-    (effects (font (size 1.27 1.27)) (justify left))
-    (property "Intersheet References" "${INTERSHEET_REFS}" (id 0) (at 13.97 -20.32 0)
-      (effects (font (size 1.27 1.27)) hide)
-    )
-  )
-  (global_label "TX0" (shape input) (at 59.69 62.23 0) (fields_autoplaced)
-    (effects (font (size 1.27 1.27)) (justify left))
-    (property "Intersheet References" "${INTERSHEET_REFS}" (id 0) (at 65.4009 62.1506 0)
-      (effects (font (size 1.27 1.27)) (justify left) hide)
-    )
-  )
-  (global_label "GND" (shape input) (at 59.69 67.31 0) (fields_autoplaced)
-    (effects (font (size 1.27 1.27)) (justify left))
-    (property "Intersheet References" "${INTERSHEET_REFS}" (id 0) (at 13.97 -12.7 0)
-      (effects (font (size 1.27 1.27)) hide)
-    )
-  )
-  (global_label "rfrx1_true" (shape input) (at 59.69 95.25 0) (fields_autoplaced)
-    (effects (font (size 1.27 1.27)) (justify left))
-    (property "Intersheet References" "${INTERSHEET_REFS}" (id 0) (at 71.2671 95.1706 0)
-      (effects (font (size 1.27 1.27)) (justify left) hide)
-    )
-  )
-  (global_label "GND" (shape input) (at 151.13 116.84 0) (fields_autoplaced)
-    (effects (font (size 1.27 1.27)) (justify left))
-    (property "Intersheet References" "${INTERSHEET_REFS}" (id 0) (at 25.4 5.08 0)
-      (effects (font (size 1.27 1.27)) hide)
-    )
-  )
-  (global_label "3V3" (shape input) (at 154.94 74.93 270) (fields_autoplaced)
-    (effects (font (size 1.27 1.27)) (justify right))
-    (property "Intersheet References" "${INTERSHEET_REFS}" (id 0) (at 85.09 149.86 0)
-      (effects (font (size 1.27 1.27)) hide)
-    )
-  )
-  (global_label "PWR" (shape input) (at 59.69 100.33 0) (fields_autoplaced)
-    (effects (font (size 1.27 1.27)) (justify left))
-    (property "Intersheet References" "${INTERSHEET_REFS}" (id 0) (at 66.0056 100.2506 0)
-      (effects (font (size 1.27 1.27)) (justify left) hide)
-    )
-  )
-  (global_label "GND" (shape input) (at 59.69 74.93 0) (fields_autoplaced)
-    (effects (font (size 1.27 1.27)) (justify left))
-    (property "Intersheet References" "${INTERSHEET_REFS}" (id 0) (at 13.97 -5.08 0)
-      (effects (font (size 1.27 1.27)) hide)
-    )
-  )
-  (global_label "GND" (shape input) (at 59.69 87.63 0) (fields_autoplaced)
-    (effects (font (size 1.27 1.27)) (justify left))
-    (property "Intersheet References" "${INTERSHEET_REFS}" (id 0) (at 13.97 -5.08 0)
-      (effects (font (size 1.27 1.27)) hide)
-    )
-  )
-  (symbol (lib_id "power:GND") (at 140.97 128.27 0) (unit 1)
-    (in_bom yes) (on_board yes)
-    (property "Reference" "#PWR01" (id 0) (at 140.97 134.62 0)
-      (effects (font (size 1.27 1.27)) hide)
-    )
-    (property "Value" "GND" (id 1) (at 141.097 132.6642 0))
-    (property "Footprint" "" (id 2) (at 140.97 128.27 0)
-      (effects (font (size 1.27 1.27)) hide)
-    )
-    (property "Datasheet" "" (id 3) (at 140.97 128.27 0)
-      (effects (font (size 1.27 1.27)) hide)
-    )
-    (pin "1")
-  )
-  (symbol (lib_id "Device:R") (at 123.19 97.79 90) (unit 1)
-    (in_bom yes) (on_board yes) (fields_autoplaced)
-    (property "Reference" "R9" (id 0) (at 123.19 93.0742 90))
-    (property "Value" "R" (id 1) (at 123.19 95.6111 90))
-    (property "Footprint" "Resistor_SMD:R_0805_2012Metric" (id 2) (at 123.19 99.568 90)
-      (effects (font (size 1.27 1.27)) hide)
-    )
-    (property "Datasheet" "~" (id 3) (at 123.19 97.79 0)
-      (effects (font (size 1.27 1.27)) hide)
-    )
-    (pin "1")
-    (pin "2")
-  )
-  (symbol (lib_id "bgt:Connector_Generic_Conn_01x20") (at 54.61 77.47 180) (unit 1)
-    (in_bom yes) (on_board yes)
-    (property "Reference" "J1" (id 0) (at 56.6928 46.355 0))
-    (property "Value" "Connector_Generic_Conn_01x20" (id 1) (at 56.6928 48.6664 0))
-    (property "Footprint" "Connector_PinHeader_2.54mm:PinHeader_1x20_P2.54mm_Vertical" (id 2) (at 54.61 77.47 0)
-      (effects (font (size 1.27 1.27)) hide)
-    )
-    (property "Datasheet" "" (id 3) (at 54.61 77.47 0)
-      (effects (font (size 1.27 1.27)) hide)
-    )
-    (pin "1")
-    (pin "10")
-    (pin "11")
-    (pin "12")
-    (pin "13")
-    (pin "14")
-    (pin "15")
-    (pin "16")
-    (pin "17")
-    (pin "18")
-    (pin "19")
-    (pin "2")
-    (pin "20")
-    (pin "3")
-    (pin "4")
-    (pin "5")
-    (pin "6")
-    (pin "7")
-    (pin "8")
-    (pin "9")
-  )
-  (symbol (lib_id "Device:C") (at 154.94 68.58 0) (unit 1)
-    (in_bom yes) (on_board yes)
-    (property "Reference" "C1" (id 0) (at 148.5392 68.58 90))
-    (property "Value" "C" (id 1) (at 150.8506 68.58 90))
-    (property "Footprint" "Capacitor_SMD:C_1206_3216Metric" (id 2) (at 155.9052 72.39 0)
-      (effects (font (size 1.27 1.27)) hide)
-    )
-    (property "Datasheet" "~" (id 3) (at 154.94 68.58 0)
-      (effects (font (size 1.27 1.27)) hide)
-    )
-    (pin "1")
-    (pin "2")
-  )
 )
